Commit message: added on gazebo

File: ernest_description/urdf/robot_core.xacro (robot description, xacro)
@@ -40,4 +40,7 @@
     </xacro:inertial_box>
   </link>
+  <gazebo reference="base_link">
+    <material>Gazebo/White</material>
+  </gazebo>
 <!-- CHASSIS -->
     <!-- REAR PART -->
@@ -60,4 +63,7 @@
     </xacro:inertial_box>
   </link>
+  <gazebo reference="back_chassis">
+    <material>Gazebo/White</material>
+  </gazebo>
     <!-- REAR WELDING -->
   <joint name="front_attatch" type="fixed">
@@ -85,4 +91,7 @@
     </xacro:inertial_box>
   </link>
+  <gazebo reference="middle_chassis">
+    <material>Gazebo/White</material>
+  </gazebo>
     <!-- STEERING JOINT -->
   <joint name="steering_joint" type="revolute">
@@ -112,4 +121,7 @@
     </xacro:inertial_box>
   </link>
+  <gazebo reference="front_chassis">
+    <material>Gazebo/White</material>
+  </gazebo>
     <!-- BOOGIE JOINT -->
   <joint name="bogie_joint" type="revolute">
@@ -140,4 +152,7 @@
       </xacro:inertial_cylinder>
     </link>
+  <gazebo reference="{wheel_prefix}_wheel_link">
+    <material>Gazebo/Black</material>
+  </gazebo>
     <!-- rolling -->
     <joint name="${wheel_prefix}_wheel" type="continuous">
