Commit message: almost imported the real rover

File: ernest_description/urdf/diff_drive_control.xacro (robot description, xacro)
@@ -5,5 +5,5 @@
           <plugin>gazebo_ros2_control/GazeboSystem</plugin>
       </hardware>
-      <joint name="rear_left_wheels">
+      <joint name="rear_left_wheel_joint">
         <command_interface name="velocity">
           <param name="min">-1</param>
@@ -14,5 +14,5 @@
         <state_interface name="effort"/>
       </joint>
-      <joint name="rear_right_wheels">
+      <joint name="rear_right_wheel_joint">
         <command_interface name="velocity">
           <param name="min">-1</param>
@@ -23,5 +23,5 @@
         <state_interface name="effort"/>
       </joint>
-      <joint name="front_left_wheels">
+      <joint name="front_left_wheel_joint">
         <command_interface name="velocity">
           <param name="min">-1</param>
@@ -32,5 +32,5 @@
         <state_interface name="effort"/>
       </joint>
-      <joint name="front_right_wheels">
+      <joint name="front_right_wheel_joint">
         <command_interface name="velocity">
           <param name="min">-1</param>

Commit message: trying to spawn the rover in gazebo

File: ernest_description/urdf/diff_drive_control.xacro (robot description, xacro)
@@ -1,7 +1,10 @@
 <?xml version="1.0"?>
-<robot xmlns:xacro="http://www.ros.org/wiki/xacro"  name="ernest">
-    <ros2_control name="diff" type="system">
+<robot xmlns:xacro="http://www.ros.org/wiki/xacro"  name="ernest_controller">
+  <xacro:macro name="ernest_system" params="name  use_gazebo:=^|false ">
+    <ros2_control name="${name}" type="system">
       <hardware>
-          <plugin>gazebo_ros2_control/GazeboSystem</plugin>
+          <xacro:if value="${use_gazebo}">
+            <plugin>gazebo_ros2_control/GazeboSystem</plugin>
+          </xacro:if>
       </hardware>
       <joint name="rear_left_wheel_joint">
@@ -23,27 +26,5 @@
         <state_interface name="effort"/>
       </joint>
-      <joint name="front_left_wheel_joint">
-        <command_interface name="velocity">
-          <param name="min">-1</param>
-          <param name="max">1</param>
-        </command_interface>
-        <state_interface name="position"/>
-        <state_interface name="velocity"/>
-        <state_interface name="effort"/>
-      </joint>
-      <joint name="front_right_wheel_joint">
-        <command_interface name="velocity">
-          <param name="min">-1</param>
-          <param name="max">1</param>
-        </command_interface>
-        <state_interface name="position"/>
-        <state_interface name="velocity"/>
-        <state_interface name="effort"/>
-      </joint>
     </ros2_control>
-    <gazebo>
-        <plugin filename="libgazebo_ros2_control.so" name="gazebo_ros2_control">
-            <parameters>$(find ernest_description)/config/diff_drive_controller_config.yaml</parameters>
-        </plugin>
-    </gazebo>
+  </xacro:macro>
 </robot>

File: ernest_description/urdf/ernest.urdf.xacro (robot description, xacro)
@@ -1,4 +1,12 @@
 <?xml version="1.0" ?>
 <robot xmlns:xacro="http://www.ros.org/wiki/xacro" name="ernest">
+<xacro:macro name="ernest" params="prefix">
+  <link name="base_link">
+  </link>
+  <joint name="frame_joint" type="fixed">
+    <origin  xyz="0 0 0.4"/>
+    <parent link="base_link"/>
+    <child link="chassis"/>
+  </joint>
   <link name="chassis">
     <inertial>
@@ -10,14 +18,14 @@
       <origin rpy="0 0 0" xyz="0 0 0"/>
       <geometry>
-        <mesh filename="package://ernest_description/meshes/chassis.dae"/>
-      </geometry>
-      <material name="">
-        <color rgba="0.752941176470588 0.752941176470588 0.752941176470588 1"/>
-      </material>
-    </visual>
-    <collision>
-      <origin rpy="0 0 0" xyz="0 0 0"/>
-      <geometry>
-        <mesh filename="package://ernest_description/meshes/chassis.dae"/>
+        <mesh filename="package://ernest_description/meshes/chassis.STL"/>
+      </geometry>
+      <material name="">
+        <color rgba="0.752941176470588 0.752941176470588 0.752941176470588 1"/>
+      </material>
+    </visual>
+    <collision>
+      <origin rpy="0 0 0" xyz="0 0 0"/>
+      <geometry>
+        <mesh filename="package://ernest_description/meshes/chassis.STL"/>
       </geometry>
     </collision>
@@ -32,14 +40,14 @@
       <origin rpy="0 0 0" xyz="0 0 0"/>
       <geometry>
-        <mesh filename="package://ernest_description/meshes/pivot.dae"/>
-      </geometry>
-      <material name="">
-        <color rgba="0.752941176470588 0.752941176470588 0.752941176470588 1"/>
-      </material>
-    </visual>
-    <collision>
-      <origin rpy="0 0 0" xyz="0 0 0"/>
-      <geometry>
-        <mesh filename="package://ernest_description/meshes/pivot.dae"/>
+        <mesh filename="package://ernest_description/meshes/pivot.STL"/>
+      </geometry>
+      <material name="">
+        <color rgba="0.752941176470588 0.752941176470588 0.752941176470588 1"/>
+      </material>
+    </visual>
+    <collision>
+      <origin rpy="0 0 0" xyz="0 0 0"/>
+      <geometry>
+        <mesh filename="package://ernest_description/meshes/pivot.STL"/>
       </geometry>
     </collision>
@@ -60,14 +68,14 @@
       <origin rpy="0 0 0" xyz="0 0 0"/>
       <geometry>
-        <mesh filename="package://ernest_description/meshes/bogie.dae"/>
-      </geometry>
-      <material name="">
-        <color rgba="0.792156862745098 0.819607843137255 0.933333333333333 1"/>
-      </material>
-    </visual>
-    <collision>
-      <origin rpy="0 0 0" xyz="0 0 0"/>
-      <geometry>
-        <mesh filename="package://ernest_description/meshes/bogie.dae"/>
+        <mesh filename="package://ernest_description/meshes/bogie.STL"/>
+      </geometry>
+      <material name="">
+        <color rgba="0.792156862745098 0.819607843137255 0.933333333333333 1"/>
+      </material>
+    </visual>
+    <collision>
+      <origin rpy="0 0 0" xyz="0 0 0"/>
+      <geometry>
+        <mesh filename="package://ernest_description/meshes/bogie.STL"/>
       </geometry>
     </collision>
@@ -88,14 +96,14 @@
       <origin rpy="0 0 0" xyz="0 0 0"/>
       <geometry>
-        <mesh filename="package://ernest_description/meshes/front_left_steer.dae"/>
-      </geometry>
-      <material name="">
-        <color rgba="0.752941176470588 0.752941176470588 0.752941176470588 1"/>
-      </material>
-    </visual>
-    <collision>
-      <origin rpy="0 0 0" xyz="0 0 0"/>
-      <geometry>
-        <mesh filename="package://ernest_description/meshes/front_left_steer.dae"/>
+        <mesh filename="package://ernest_description/meshes/front_left_steer.STL"/>
+      </geometry>
+      <material name="">
+        <color rgba="0.752941176470588 0.752941176470588 0.752941176470588 1"/>
+      </material>
+    </visual>
+    <collision>
+      <origin rpy="0 0 0" xyz="0 0 0"/>
+      <geometry>
+        <mesh filename="package://ernest_description/meshes/front_left_steer.STL"/>
       </geometry>
     </collision>
@@ -116,14 +124,14 @@
       <origin rpy="0 0 0" xyz="0 0 0"/>
       <geometry>
-        <mesh filename="package://ernest_description/meshes/front_left_wheel.dae"/>
-      </geometry>
-      <material name="">
-        <color rgba="0.792156862745098 0.819607843137255 0.933333333333333 1"/>
-      </material>
-    </visual>
-    <collision>
-      <origin rpy="0 0 0" xyz="0 0 0"/>
-      <geometry>
-        <mesh filename="package://ernest_description/meshes/front_left_wheel.dae"/>
+        <mesh filename="package://ernest_description/meshes/front_left_wheel.STL"/>
+      </geometry>
+      <material name="">
+        <color rgba="0.792156862745098 0.819607843137255 0.933333333333333 1"/>
+      </material>
+    </visual>
+    <collision>
+      <origin rpy="0 0 0" xyz="0 0 0"/>
+      <geometry>
+        <mesh filename="package://ernest_description/meshes/front_left_wheel.STL"/>
       </geometry>
     </collision>
@@ -144,14 +152,14 @@
       <origin rpy="0 0 0" xyz="0 0 0"/>
       <geometry>
-        <mesh filename="package://ernest_description/meshes/front_right_steer.dae"/>
-      </geometry>
-      <material name="">
-        <color rgba="0.752941176470588 0.752941176470588 0.752941176470588 1"/>
-      </material>
-    </visual>
-    <collision>
-      <origin rpy="0 0 0" xyz="0 0 0"/>
-      <geometry>
-        <mesh filename="package://ernest_description/meshes/front_right_steer.dae"/>
+        <mesh filename="package://ernest_description/meshes/front_right_steer.STL"/>
+      </geometry>
+      <material name="">
+        <color rgba="0.752941176470588 0.752941176470588 0.752941176470588 1"/>
+      </material>
+    </visual>
+    <collision>
+      <origin rpy="0 0 0" xyz="0 0 0"/>
+      <geometry>
+        <mesh filename="package://ernest_description/meshes/front_right_steer.STL"/>
       </geometry>
     </collision>
@@ -172,14 +180,14 @@
       <origin rpy="0 0 0" xyz="0 0 0"/>
       <geometry>
-        <mesh filename="package://ernest_description/meshes/front_right_wheel.dae"/>
-      </geometry>
-      <material name="">
-        <color rgba="0.792156862745098 0.819607843137255 0.933333333333333 1"/>
-      </material>
-    </visual>
-    <collision>
-      <origin rpy="0 0 0" xyz="0 0 0"/>
-      <geometry>
-        <mesh filename="package://ernest_description/meshes/front_right_wheel.dae"/>
+        <mesh filename="package://ernest_description/meshes/front_right_wheel.STL"/>
+      </geometry>
+      <material name="">
+        <color rgba="0.792156862745098 0.819607843137255 0.933333333333333 1"/>
+      </material>
+    </visual>
+    <collision>
+      <origin rpy="0 0 0" xyz="0 0 0"/>
+      <geometry>
+        <mesh filename="package://ernest_description/meshes/front_right_wheel.STL"/>
       </geometry>
     </collision>
@@ -200,14 +208,14 @@
       <origin rpy="0 0 0" xyz="0 0 0"/>
       <geometry>
-        <mesh filename="package://ernest_description/meshes/rear_right_steer.dae"/>
-      </geometry>
-      <material name="">
-        <color rgba="0.752941176470588 0.752941176470588 0.752941176470588 1"/>
-      </material>
-    </visual>
-    <collision>
-      <origin rpy="0 0 0" xyz="0 0 0"/>
-      <geometry>
-        <mesh filename="package://ernest_description/meshes/rear_right_steer.dae"/>
+        <mesh filename="package://ernest_description/meshes/rear_right_steer.STL"/>
+      </geometry>
+      <material name="">
+        <color rgba="0.752941176470588 0.752941176470588 0.752941176470588 1"/>
+      </material>
+    </visual>
+    <collision>
+      <origin rpy="0 0 0" xyz="0 0 0"/>
+      <geometry>
+        <mesh filename="package://ernest_description/meshes/rear_right_steer.STL"/>
       </geometry>
     </collision>
@@ -228,14 +236,14 @@
       <origin rpy="0 0 0" xyz="0 0 0"/>
       <geometry>
-        <mesh filename="package://ernest_description/meshes/rear_right_wheel.dae"/>
-      </geometry>
-      <material name="">
-        <color rgba="0.792156862745098 0.819607843137255 0.933333333333333 1"/>
-      </material>
-    </visual>
-    <collision>
-      <origin rpy="0 0 0" xyz="0 0 0"/>
-      <geometry>
-        <mesh filename="package://ernest_description/meshes/rear_right_wheel.dae"/>
+        <mesh filename="package://ernest_description/meshes/rear_right_wheel.STL"/>
+      </geometry>
+      <material name="">
+        <color rgba="0.792156862745098 0.819607843137255 0.933333333333333 1"/>
+      </material>
+    </visual>
+    <collision>
+      <origin rpy="0 0 0" xyz="0 0 0"/>
+      <geometry>
+        <mesh filename="package://ernest_description/meshes/rear_right_wheel.STL"/>
       </geometry>
     </collision>
@@ -256,14 +264,14 @@
       <origin rpy="0 0 0" xyz="0 0 0"/>
       <geometry>
-        <mesh filename="package://ernest_description/meshes/rear_left_steer.dae"/>
-      </geometry>
-      <material name="">
-        <color rgba="0.752941176470588 0.752941176470588 0.752941176470588 1"/>
-      </material>
-    </visual>
-    <collision>
-      <origin rpy="0 0 0" xyz="0 0 0"/>
-      <geometry>
-        <mesh filename="package://ernest_description/meshes/rear_left_steer.dae"/>
+        <mesh filename="package://ernest_description/meshes/rear_left_steer.STL"/>
+      </geometry>
+      <material name="">
+        <color rgba="0.752941176470588 0.752941176470588 0.752941176470588 1"/>
+      </material>
+    </visual>
+    <collision>
+      <origin rpy="0 0 0" xyz="0 0 0"/>
+      <geometry>
+        <mesh filename="package://ernest_description/meshes/rear_left_steer.STL"/>
       </geometry>
     </collision>
@@ -284,14 +292,14 @@
       <origin rpy="0 0 0" xyz="0 0 0"/>
       <geometry>
-        <mesh filename="package://ernest_description/meshes/rear_left_wheel.dae"/>
-      </geometry>
-      <material name="">
-        <color rgba="0.792156862745098 0.819607843137255 0.933333333333333 1"/>
-      </material>
-    </visual>
-    <collision>
-      <origin rpy="0 0 0" xyz="0 0 0"/>
-      <geometry>
-        <mesh filename="package://ernest_description/meshes/rear_left_wheel.dae"/>
+        <mesh filename="package://ernest_description/meshes/rear_left_wheel.STL"/>
+      </geometry>
+      <material name="">
+        <color rgba="0.792156862745098 0.819607843137255 0.933333333333333 1"/>
+      </material>
+    </visual>
+    <collision>
+      <origin rpy="0 0 0" xyz="0 0 0"/>
+      <geometry>
+        <mesh filename="package://ernest_description/meshes/rear_left_wheel.STL"/>
       </geometry>
     </collision>
@@ -303,2 +311,4 @@
     <axis xyz="0 0 1"/>
   </joint>
+</xacro:macro>
+</robot>

File: ernest_description/urdf/ernest_system.urdf.xacro (robot description, xacro)
@@ -1,5 +1,24 @@
 <?xml version="1.0"?>
-<robot xmlns:xacro="http://www.ros.org/wiki/xacro"  name="ernest">
-    <xacro:include filename="asterix.urdf.xacro" />
-  <!--  <xacro:include filename="diff_drive_control.xacro" /> -->
+<robot xmlns:xacro="http://www.ros.org/wiki/xacro"  name="ernest_system">
+  <!-- Enable setting arguments from the launch file -->
+  <xacro:arg name="use_fake_hardware" default="true" />
+  <xacro:arg name="use_gazebo" default="true" />
+  <xacro:arg name="use_lowpoly" default="true" />
+  <xacro:include filename="$(find ernest_description)/urdf/ernest.urdf.xacro" />
+  <xacro:include filename="$(find ernest_description)/urdf/robot_core.urdf.xacro" />
+  <!-- Import stm ros2_control description -->
+  <xacro:include filename="$(find ernest_description)/urdf/diff_drive_control.xacro"/>
+  <xacro:include filename="$(find ernest_description)/gazebo/ernest_gazebo.xacro" />
+  <xacro:ernest_system
+    name="ErnestSystem"
+    use_gazebo="$(arg use_gazebo)"/>
+  <xacro:if value="$(arg use_gazebo)">
+    <xacro:ernest_gazebo prefix=""/>
+  </xacro:if>
+  <xacro:if value="$(arg use_lowpoly)">
+    <xacro:robot_core prefix=""/>
+  </xacro:if>
+  <xacro:unless value="$(arg use_lowpoly)">
+    <xacro:ernest prefix=""/>
+  </xacro:unless>
 </robot>

File: ernest_description/urdf/robot_core.urdf.xacro (robot description, xacro)
@@ -1,4 +1,5 @@
 <?xml version="1.0"?>
-<robot xmlns:xacro="http://www.ros.org/wiki/xacro" name="ernest">
+<robot xmlns:xacro="http://www.ros.org/wiki/xacro" name="ernest_lowpoly">
+<xacro:macro name="robot_core" params="prefix">
   <xacro:include filename="inertial_macros.xacro"/>
   <xacro:property name="body_width" value="0.318"/>
@@ -21,6 +22,13 @@
       <color rgba="0 0 0 1"/>
   </material>
+  <link name="${prefix}base_link">
+  </link>
+  <joint name="${prefix}frame_joint" type="fixed">
+    <origin  xyz="0 0 0"/>
+    <parent link="base_link"/>
+    <child link="chassis"/>
+  </joint>
 <!-- BASE LINK -->
-  <link name="base_link">
+  <link name="${prefix}chassis">
     <visual>
       <origin xyz="0 0 0" rpy="0 0 0"/>
@@ -40,10 +48,7 @@
     </xacro:inertial_box>
   </link>
-  <gazebo reference="base_link">
-    <material>Gazebo/White</material>
-  </gazebo>
 <!-- CHASSIS -->
     <!-- REAR PART -->
-  <link name="back_chassis">
+  <link name="${prefix}back_chassis">
     <visual>
       <geometry>
@@ -63,15 +68,12 @@
     </xacro:inertial_box>
   </link>
-  <gazebo reference="back_chassis">
-    <material>Gazebo/White</material>
-  </gazebo>
     <!-- REAR WELDING -->
-  <joint name="front_attatch" type="fixed">
-    <parent link="base_link"/>
+  <joint name="${prefix}front_attatch" type="fixed">
+    <parent link="chassis"/>
     <child link="back_chassis"/>
     <origin xyz="${chassis_thickness/-2} 0 0"/>
   </joint>
     <!-- MIDDLE PART -->
-  <link name="middle_chassis">
+  <link name="${prefix}pivot">
     <visual>
       <geometry>
@@ -91,17 +93,14 @@
     </xacro:inertial_box>
   </link>
-  <gazebo reference="middle_chassis">
-    <material>Gazebo/White</material>
-  </gazebo>
     <!-- STEERING JOINT -->
-  <joint name="steering_joint" type="fixed">
-    <!-- <axis xyz="0 0 -1"/> -->
-     <!-- <limit effort="50" lower="-1.571" upper="1.571" velocity="30"/> -->
+  <joint name="${prefix}pivot_joint" type="revolute">
+    <axis xyz="0 0 -1"/>
+    <limit effort="50" lower="-1.571" upper="1.571" velocity="30"/>
     <parent link="back_chassis"/>
-    <child link="middle_chassis"/>
+    <child link="pivot"/>
     <origin xyz="${-1*middle_chassis_length} 0 0"/>
   </joint>
     <!-- FRONT PART -->
-  <link name="front_chassis">
+  <link name="${prefix}bogie">
     <visual>
       <geometry>
@@ -121,18 +120,15 @@
     </xacro:inertial_box>
   </link>
-  <gazebo reference="front_chassis">
-    <material>Gazebo/White</material>
-  </gazebo>
     <!-- BOOGIE JOINT -->
-  <joint name="bogie_joint" type="revolute">
+  <joint name="${prefix}bogie_joint" type="revolute">
     <axis xyz="0 0 1"/>
     <limit effort="50" lower="-1.571" upper="1.571" velocity="30"/>
-    <parent link="middle_chassis"/>
-    <child link="front_chassis"/>
+    <parent link="pivot"/>
+    <child link="bogie"/>
     <origin xyz="${body_length/-2} 0 0" rpy="0 ${-pi/2} 0"/>
   </joint>
 <!-- WHEELS-->
   <xacro:macro name="wheel" params="wheel_prefix flip parent *joint_pose">
-    <link name="${wheel_prefix}_wheel_link">
+    <link name="${wheel_prefix}_wheel">
       <visual>
         <origin xyz="0 0 0" rpy="0 0 ${flip*pi/2}" />
@@ -152,11 +148,8 @@
       </xacro:inertial_cylinder>
     </link>
-  <gazebo reference="{wheel_prefix}_wheel_link">
-    <material>Gazebo/Black</material>
-  </gazebo>
     <!-- rolling -->
-    <joint name="${wheel_prefix}_wheels" type="continuous">
+    <joint name="${wheel_prefix}_wheel_joint" type="continuous">
       <parent link="${parent}"/>
-      <child link="${wheel_prefix}_wheel_link"/>
+      <child link="${wheel_prefix}_wheel"/>
       <xacro:insert_block name="joint_pose"/>
       <axis xyz="0 0 1" rpy="0 0 0" />
@@ -166,20 +159,21 @@
       <limit effort="50" lower="-1.571" upper="1.571" velocity="30"/>
       <parent link="${parent}"/>
-      <child link="${wheel_prefix}_wheel_link"/>
+      <child link="${wheel_prefix}_wheel"/>
       <xacro:insert_block name="joint_pose"/>
       <axis xyz="0 0 -1" rpy="0 0 0" />
     </joint>
   </xacro:macro>
-  <xacro:wheel wheel_prefix="front_left" flip="-1" parent="front_chassis">
+  <xacro:wheel wheel_prefix="${prefix}front_left" flip="-1" parent="${prefix}bogie">
     <origin xyz="0 ${-body_width/2} -.009" rpy="${pi/2} 0 0" />
   </xacro:wheel>
-  <xacro:wheel wheel_prefix="front_right" flip="1" parent="front_chassis">
+  <xacro:wheel wheel_prefix="${prefix}front_right" flip="1" parent="${prefix}bogie">
     <origin xyz="0 ${body_width/2} -.009" rpy="${pi/2} 0 0" />
   </xacro:wheel>
-  <xacro:wheel wheel_prefix="rear_left" flip="-1" parent="base_link">
+  <xacro:wheel wheel_prefix="${prefix}rear_left" flip="-1" parent="${prefix}chassis">
     <origin xyz="0 ${-body_width/2} -.009" rpy="${pi/2} 0 0" />
   </xacro:wheel>
-  <xacro:wheel wheel_prefix="rear_right" flip="1" parent="base_link">
+  <xacro:wheel wheel_prefix="${prefix}rear_right" flip="1" parent="${prefix}chassis">
     <origin xyz="0 ${body_width/2} -.009" rpy="${pi/2} 0 0" />
   </xacro:wheel>
+</xacro:macro>
 </robot>

Commit message: added the model to gazebo

File: ernest_description/urdf/diff_drive_control.xacro (robot description, xacro)
@@ -8,5 +8,5 @@
           </xacro:if>
       </hardware>
-      <joint name="rear_left_wheel_joint">
+      <joint name="rear_left_wheel_steer">
         <command_interface name="velocity">
           <param name="min">-1</param>
@@ -15,7 +15,6 @@
         <state_interface name="position"/>
         <state_interface name="velocity"/>
-        <state_interface name="effort"/>
       </joint>
-      <joint name="rear_right_wheel_joint">
+      <joint name="rear_right_wheel_steer">
         <command_interface name="velocity">
           <param name="min">-1</param>
@@ -24,5 +23,20 @@
         <state_interface name="position"/>
         <state_interface name="velocity"/>
-        <state_interface name="effort"/>
+      </joint>
+      <joint name="front_left_wheel_steer">
+        <command_interface name="velocity">
+          <param name="min">-1</param>
+          <param name="max">1</param>
+        </command_interface>
+        <state_interface name="position"/>
+        <state_interface name="velocity"/>
+      </joint>
+      <joint name="front_right_wheel_steer">
+        <command_interface name="velocity">
+          <param name="min">-1</param>
+          <param name="max">1</param>
+        </command_interface>
+        <state_interface name="position"/>
+        <state_interface name="velocity"/>
       </joint>
     </ros2_control>

File: ernest_description/urdf/robot_core.urdf.xacro (robot description, xacro)
@@ -148,11 +148,4 @@
       </xacro:inertial_cylinder>
     </link>
-    <!-- rolling -->
-    <joint name="${wheel_prefix}_wheel_joint" type="continuous">
-      <parent link="${parent}"/>
-      <child link="${wheel_prefix}_wheel"/>
-      <xacro:insert_block name="joint_pose"/>
-      <axis xyz="0 0 1" rpy="0 0 0" />
-    </joint>
     <!-- steering -->
     <joint name="${wheel_prefix}_wheel_steer" type="revolute">
@@ -162,4 +155,11 @@
       <xacro:insert_block name="joint_pose"/>
       <axis xyz="0 0 -1" rpy="0 0 0" />
+    </joint>
+    <!-- rolling -->
+    <joint name="${wheel_prefix}_wheel_joint" type="continuous">
+      <parent link="${parent}"/>
+      <child link="${wheel_prefix}_wheel"/>
+      <xacro:insert_block name="joint_pose"/>
+      <axis xyz="0 0 1" rpy="0 0 0" />
     </joint>
   </xacro:macro>
