Commit message: started adding vel controller

File: ernest_description/urdf/joint_traj_controller.xacro (robot description, xacro)
@@ -48,4 +48,20 @@
         <state_interface name="velocity"/>
       </joint>
+      <joint name="rear_right_wheel_joint">
+        <command_interface name="velocity">
+          <param name="min">-2</param>
+          <param name="max">2</param>
+        </command_interface>
+        <state_interface name="position"/>
+        <state_interface name="velocity"/>
+      </joint>
+      <joint name="rear_left_wheel_joint">
+        <command_interface name="velocity">
+          <param name="min">--2</param>
+          <param name="max">2</param>
+        </command_interface>
+        <state_interface name="position"/>
+        <state_interface name="velocity"/>
+      </joint>
     </ros2_control>
   </xacro:macro>
