Commit message: completed both controller level

File: description/urdf/effort_joint.xacro (robot description, xacro)
@@ -1,18 +1,85 @@
 <?xml version="1.0"?>
 <robot xmlns:xacro="http://www.ros.org/wiki/xacro"  name="ernest_controller">
-  <xacro:macro name="joint_traj_controller">
+  <xacro:macro name="effort_joint">
     <ros2_control name="Joint Control" type="system">
       <hardware>
           <plugin>gazebo_ros2_control/GazeboSystem</plugin>
       </hardware>
-     <!-- <joint name="pivot_joint">
-        <command_interface name="effort"/>
+      <joint name="front_left_wheel_joint">
+        <command_interface name="effort">
+          <param name="min">-100</param>
+          <param name="max">100</param>
+        </command_interface>
+        <state_interface name="position"/>
+        <state_interface name="velocity"/>
         <state_interface name="effort"/>
       </joint>
-    </ros2_control> -->
+      <joint name="front_right_wheel_joint">
+        <command_interface name="effort">
+          <param name="min">-100</param>
+          <param name="max">100</param>
+        </command_interface>
+        <state_interface name="position"/>
+        <state_interface name="velocity"/>
+        <state_interface name="effort"/>
+      </joint>
+      <joint name="rear_left_wheel_joint">
+        <command_interface name="effort">
+          <param name="min">-100</param>
+          <param name="max">100</param>
+        </command_interface>
+        <state_interface name="position"/>
+        <state_interface name="velocity"/>
+        <state_interface name="effort"/>
+      </joint>
+      <joint name="rear_right_wheel_joint">
+        <command_interface name="effort">
+          <param name="min">-100</param>
+          <param name="max">100</param>
+        </command_interface>
+        <state_interface name="position"/>
+        <state_interface name="velocity"/>
+        <state_interface name="effort"/>
+      </joint>
+      <joint name="front_left_steer_joint">
+        <command_interface name="effort">
+          <param name="min">-100</param>
+          <param name="max">100</param>
+        </command_interface>
+        <state_interface name="position"/>
+        <state_interface name="velocity"/>
+        <state_interface name="effort"/>
+      </joint>
+      <joint name="front_right_steer_joint">
+        <command_interface name="effort">
+          <param name="min">-100</param>
+          <param name="max">100</param>
+        </command_interface>
+        <state_interface name="position"/>
+        <state_interface name="velocity"/>
+        <state_interface name="effort"/>
+      </joint>
+      <joint name="rear_left_steer_joint">
+        <command_interface name="effort">
+          <param name="min">-100</param>
+          <param name="max">100</param>
+        </command_interface>
+        <state_interface name="position"/>
+        <state_interface name="velocity"/>
+        <state_interface name="effort"/>
+      </joint>
+      <joint name="rear_right_steer_joint">
+        <command_interface name="effort">
+          <param name="min">-100</param>
+          <param name="max">100</param>
+        </command_interface>
+        <state_interface name="position"/>
+        <state_interface name="velocity"/>
+        <state_interface name="effort"/>
+      </joint>
       <joint name="pivot_joint">
-        <command_interface name="position">
-          <param name="min">-1000</param>
-          <param name="max">1000</param>
+        <command_interface name="effort">
+          <param name="min">-100</param>
+          <param name="max">100</param>
         </command_interface>
         <state_interface name="position"/>

File: description/urdf/ernest.urdf.xacro (robot description, xacro)
@@ -52,5 +52,5 @@
   </link>
   <joint name="pivot_joint" type="revolute">
-    <limit effort="5.0" lower="-0.8" upper="0.8" velocity="2"/>
+    <limit effort="100.0" lower="-0.8" upper="0.8" velocity="2"/>
     <origin rpy="0 0 3.13911747329568" xyz="0 0.4015 -0.00700000000000001"/>
     <parent link="chassis"/>
@@ -80,5 +80,5 @@
   </link>
   <joint name="bogie_joint" type="revolute">
-    <limit effort="1000" lower="-1" upper="1" velocity="30"/>
+    <limit effort="100" lower="-1" upper="1" velocity="30"/>
     <origin rpy="1.5707963267949 0.000529942236827729 0" xyz="0 -0.101800622452903 -0.0640000000000083"/>
     <parent link="pivot"/>
@@ -107,5 +107,5 @@
   </link>
   <joint name="front_left_steer_joint" type="revolute">
-    <limit effort="50" lower="-0.8" upper="0.8" velocity="30"/>
+    <limit effort="100" lower="-1.57" upper="1.57" velocity="30"/>
     <origin rpy="-1.5707963267949 0.0208107531087718 0" xyz="0.399593578400315 0.05 0.0507993775470971"/>
     <parent link="bogie"/>
@@ -160,5 +160,5 @@
   </link>
   <joint name="front_right_steer_joint" type="revolute">
-    <limit effort="50" lower="-0.8" upper="0.8" velocity="30"/>
+    <limit effort="100" lower="-1.57" upper="1.57" velocity="30"/>
     <origin rpy="-1.57079632679545 -1.56850410535828 0" xyz="-0.399593578400314 0.05 0.0507993775470972"/>
     <parent link="bogie"/>
@@ -213,5 +213,5 @@
   </link>
   <joint name="rear_right_steer_joint" type="revolute">
-    <limit effort="50" lower="-0.8" upper="0.8" velocity="30"/>
+    <limit effort="100" lower="-1.57" upper="1.57" velocity="30"/>
     <origin rpy="0 0 0" xyz="0.4038086578651 -0.313808657865102 -0.01666"/>
     <parent link="chassis"/>
@@ -266,5 +266,5 @@
   </link>
   <joint name="rear_left_steer_joint" type="revolute">
-    <limit effort="50" lower="-0.8" upper="0.8" velocity="30"/>
+    <limit effort="100" lower="-1.57" upper="1.57" velocity="30"/>
     <origin rpy="0 0 -1.56733797587802" xyz="-0.403808657865099 -0.313808657865101 -0.01666"/>
     <parent link="chassis"/>

File: description/urdf/ernest_gazebo.xacro (robot description, xacro)
@@ -4,5 +4,5 @@
   <gazebo>
       <plugin filename="libgazebo_ros2_control.so" name="gazebo_ros2_control">
-        <parameters>$(find bringup)/config/joint_controller_config.yaml</parameters>
+        <parameters>$(find bringup)/config/effort_controller_config.yaml</parameters>
       </plugin>
   </gazebo>
@@ -11,10 +11,9 @@
     <plugin filename="libgazebo_ros_p3d.so" name="gazebo_ros_p3d">
       <ros>
-          <namespace>p3d</namespace>
           <remapping>odom:=odom</remapping>
       </ros>
       <frame_name>map</frame_name>
       <body_name>base_link</body_name>
-      <update_rate>10000.0</update_rate>
+      <update_rate>1000.0</update_rate>
       <gaussian_noise>0.0</gaussian_noise>
     </plugin>

File: description/urdf/ernest_system.urdf.xacro (robot description, xacro)
@@ -4,9 +4,9 @@
   <xacro:include filename="$(find description)/urdf/ernest.urdf.xacro"/>
   <!-- Import controller -->
-  <xacro:include filename="$(find description)/urdf/joint_traj_controller.xacro"/>
+  <xacro:include filename="$(find description)/urdf/effort_joint.xacro"/>
   <!-- Import gazebo references + pose -->
   <xacro:include filename="$(find description)/urdf/ernest_gazebo.xacro" />
   <xacro:ernest_gazebo/>
   <xacro:ernest/>
-  <xacro:joint_traj_controller/>
+  <xacro:effort_joint/>
 </robot>

Commit message: pid calibrated and starting to adding the odom to tf

File: description/urdf/effort_joint.xacro (robot description, xacro)
@@ -87,4 +87,9 @@
         <state_interface name="effort"/>
       </joint>
+      <joint name="bogie_joint">
+        <state_interface name="position"/>
+        <state_interface name="velocity"/>
+        <state_interface name="effort"/>
+      </joint>
     </ros2_control>
   </xacro:macro>

File: description/urdf/ernest.urdf.xacro (robot description, xacro)
@@ -20,5 +20,5 @@
       <origin rpy="0 0 0" xyz="0 0 0"/>
       <geometry>
-        <mesh filename="package://description/meshes/chassis.STL"/>
+        <mesh filename="file://$(find description)/meshes/chassis.STL"/>
       </geometry>
       <material name="white"/>
@@ -27,5 +27,5 @@
       <origin rpy="0 0 0" xyz="0 0 0"/>
       <geometry>
-        <mesh filename="package://description/meshes/chassis.STL"/>
+        <mesh filename="file://$(find description)/meshes/chassis.STL"/>
       </geometry>
     </collision>
@@ -40,17 +40,17 @@
       <origin rpy="0 0 0" xyz="0 0 0"/>
       <geometry>
-        <mesh filename="package://description/meshes/pivot.STL"/>
-      </geometry>
-      <material name="black"/>
-    </visual>
-    <collision>
-      <origin rpy="0 0 0" xyz="0 0 0"/>
-      <geometry>
-        <mesh filename="package://description/meshes/pivot.STL"/>
+        <mesh filename="file://$(find description)/meshes/pivot.STL"/>
+      </geometry>
+      <material name="black"/>
+    </visual>
+    <collision>
+      <origin rpy="0 0 0" xyz="0 0 0"/>
+      <geometry>
+        <mesh filename="file://$(find description)/meshes/pivot.STL"/>
       </geometry>
     </collision>
   </link>
   <joint name="pivot_joint" type="revolute">
-    <limit effort="100.0" lower="-0.8" upper="0.8" velocity="2"/>
+    <limit effort="100.0" lower="-0.8" upper="0.8" velocity="10"/>
     <origin rpy="0 0 3.13911747329568" xyz="0 0.4015 -0.00700000000000001"/>
     <parent link="chassis"/>
@@ -68,5 +68,5 @@
       <origin rpy="0 0 0" xyz="0 0 0"/>
       <geometry>
-        <mesh filename="package://description/meshes/bogie.STL"/>
+        <mesh filename="file://$(find description)/meshes/bogie.STL"/>
       </geometry>
       <material name="white"/>
@@ -75,5 +75,5 @@
       <origin rpy="0 0 0" xyz="0 0 0"/>
       <geometry>
-        <mesh filename="package://description/meshes/bogie.STL"/>
+        <mesh filename="file://$(find description)/meshes/bogie.STL"/>
       </geometry>
     </collision>
@@ -95,12 +95,12 @@
       <origin rpy="0 0 0" xyz="0 0 0"/>
       <geometry>
-        <mesh filename="package://description/meshes/front_left_steer.STL"/>
-      </geometry>
-      <material name="black"/>
-    </visual>
-    <collision>
-      <origin rpy="0 0 0" xyz="0 0 0"/>
-      <geometry>
-        <mesh filename="package://description/meshes/front_left_steer.STL"/>
+        <mesh filename="file://$(find description)/meshes/front_left_steer.STL"/>
+      </geometry>
+      <material name="black"/>
+    </visual>
+    <collision>
+      <origin rpy="0 0 0" xyz="0 0 0"/>
+      <geometry>
+        <mesh filename="file://$(find description)/meshes/front_left_steer.STL"/>
       </geometry>
     </collision>
@@ -123,5 +123,5 @@
       <origin rpy="0 0 0" xyz="0 0 0"/>
       <geometry>
-        <mesh filename="package://description/meshes/front_left_wheel.STL"/>
+        <mesh filename="file://$(find description)/meshes/front_left_wheel.STL"/>
       </geometry>
       <material name="grey"/>
@@ -130,5 +130,5 @@
       <origin rpy="0 0 0" xyz="0 0 0.0"/>
       <geometry>
-          <mesh filename="package://description/meshes/front_left_wheel.STL"/>
+          <mesh filename="file://$(find description)/meshes/front_left_wheel.STL"/>
       </geometry>
     </collision>
@@ -148,12 +148,12 @@
       <origin rpy="0 0 0" xyz="0 0 0"/>
       <geometry>
-        <mesh filename="package://description/meshes/front_right_steer.STL"/>
-      </geometry>
-      <material name="black"/>
-    </visual>
-    <collision>
-      <origin rpy="0 0 0" xyz="0 0 0"/>
-      <geometry>
-        <mesh filename="package://description/meshes/front_right_steer.STL"/>
+        <mesh filename="file://$(find description)/meshes/front_right_steer.STL"/>
+      </geometry>
+      <material name="black"/>
+    </visual>
+    <collision>
+      <origin rpy="0 0 0" xyz="0 0 0"/>
+      <geometry>
+        <mesh filename="file://$(find description)/meshes/front_right_steer.STL"/>
       </geometry>
     </collision>
@@ -176,5 +176,5 @@
       <origin rpy="0 0 0" xyz="0 0 0"/>
       <geometry>
-        <mesh filename="package://description/meshes/front_right_wheel.STL"/>
+        <mesh filename="file://$(find description)/meshes/front_right_wheel.STL"/>
       </geometry>
       <material name="grey"/>
@@ -183,5 +183,5 @@
       <origin rpy="0 0 0" xyz="0 0 0.0"/>
       <geometry>
-        <mesh filename="package://description/meshes/front_right_wheel.STL"/>
+        <mesh filename="file://$(find description)/meshes/front_right_wheel.STL"/>
       </geometry>
     </collision>
@@ -201,12 +201,12 @@
       <origin rpy="0 0 0" xyz="0 0 0"/>
       <geometry>
-        <mesh filename="package://description/meshes/rear_right_steer.STL"/>
-      </geometry>
-      <material name="black"/>
-    </visual>
-    <collision>
-      <origin rpy="0 0 0" xyz="0 0 0"/>
-      <geometry>
-        <mesh filename="package://description/meshes/rear_right_steer.STL"/>
+        <mesh filename="file://$(find description)/meshes/rear_right_steer.STL"/>
+      </geometry>
+      <material name="black"/>
+    </visual>
+    <collision>
+      <origin rpy="0 0 0" xyz="0 0 0"/>
+      <geometry>
+        <mesh filename="file://$(find description)/meshes/rear_right_steer.STL"/>
       </geometry>
     </collision>
@@ -229,5 +229,5 @@
       <origin rpy="0 0 0" xyz="0 0 0"/>
       <geometry>
-        <mesh filename="package://description/meshes/rear_right_wheel.STL"/>
+        <mesh filename="file://$(find description)/meshes/rear_right_wheel.STL"/>
       </geometry>
       <material name="grey"/>
@@ -236,5 +236,5 @@
       <origin rpy="0 0 0" xyz="0 0 0.0"/>
       <geometry>
-        <mesh filename="package://description/meshes/rear_right_wheel.STL"/>
+        <mesh filename="file://$(find description)/meshes/rear_right_wheel.STL"/>
       </geometry>
     </collision>
@@ -254,12 +254,12 @@
       <origin rpy="0 0 0" xyz="0 0 0"/>
       <geometry>
-        <mesh filename="package://description/meshes/rear_left_steer.STL"/>
-      </geometry>
-      <material name="black"/>
-    </visual>
-    <collision>
-      <origin rpy="0 0 0" xyz="0 0 0"/>
-      <geometry>
-        <mesh filename="package://description/meshes/rear_left_steer.STL"/>
+        <mesh filename="file://$(find description)/meshes/rear_left_steer.STL"/>
+      </geometry>
+      <material name="black"/>
+    </visual>
+    <collision>
+      <origin rpy="0 0 0" xyz="0 0 0"/>
+      <geometry>
+        <mesh filename="file://$(find description)/meshes/rear_left_steer.STL"/>
       </geometry>
     </collision>
@@ -282,5 +282,5 @@
       <origin rpy="0 0 0" xyz="0 0 0"/>
       <geometry>
-        <mesh filename="package://description/meshes/rear_left_wheel.STL"/>
+        <mesh filename="file://$(find description)/meshes/rear_left_wheel.STL"/>
       </geometry>
       <material name="grey"/>
@@ -289,5 +289,5 @@
       <origin rpy="0 0 0" xyz="0 0 0.0"/>
       <geometry>
-        <mesh filename="package://description/meshes/rear_left_wheel.STL"/>
+        <mesh filename="file://$(find description)/meshes/rear_left_wheel.STL"/>
       </geometry>
     </collision>

File: description/urdf/ernest_gazebo.xacro (robot description, xacro)
@@ -141,7 +141,6 @@
   <gazebo reference="front_left_wheel">
     <material>Gazebo/Grey</material>
-    <mu1>1.0</mu1>
-    <mu2>1.0</mu2>
-    <fdir1>1 0 0</fdir1>
+    <mu1>2.0</mu1>
+    <mu2>2.0</mu2>
     <kp>10000000.0</kp>
     <kd>10.0</kd>
@@ -151,7 +150,6 @@
   <gazebo reference="front_right_wheel">
     <material>Gazebo/Grey</material>
-    <mu1>1.0</mu1>
-    <mu2>1.0</mu2>
-    <fdir1>1 0 0</fdir1>
+    <mu1>2.0</mu1>
+    <mu2>2.0</mu2>
     <kp>10000000.0</kp>
     <kd>10.0</kd>
@@ -161,6 +159,6 @@
   <gazebo reference="rear_left_wheel">
     <material>Gazebo/Grey</material>
-    <mu1>1.0</mu1>
-    <mu2>1.0</mu2>
+    <mu1>2.0</mu1>
+    <mu2>2.0</mu2>
     <kp>10000000.0</kp>
     <kd>10.0</kd>
@@ -170,6 +168,6 @@
   <gazebo reference="rear_right_wheel">
     <material>Gazebo/Grey</material>
-    <mu1>1.0</mu1>
-    <mu2>1.0</mu2>
+    <mu1>2.0</mu1>
+    <mu2>2.0</mu2>
     <kp>10000000.0</kp>
     <kd>10.0</kd>
