Commit message: added odometry and renamed packages

File: description/urdf/ernest.urdf.xacro (robot description, xacro)
@@ -18,14 +18,14 @@
       <origin rpy="0 0 0" xyz="0 0 0"/>
       <geometry>
-        <mesh filename="package://ernest_description/meshes/chassis.STL"/>
-      </geometry>
-      <material name="">
-        <color rgba="0.752941176470588 0.752941176470588 0.752941176470588 1"/>
-      </material>
-    </visual>
-    <collision>
-      <origin rpy="0 0 0" xyz="0 0 0"/>
-      <geometry>
-        <mesh filename="package://ernest_description/meshes/chassis.STL"/>
+        <mesh filename="package://description/meshes/chassis.STL"/>
+      </geometry>
+      <material name="">
+        <color rgba="0.752941176470588 0.752941176470588 0.752941176470588 1"/>
+      </material>
+    </visual>
+    <collision>
+      <origin rpy="0 0 0" xyz="0 0 0"/>
+      <geometry>
+        <mesh filename="package://description/meshes/chassis.STL"/>
       </geometry>
     </collision>
@@ -40,14 +40,14 @@
       <origin rpy="0 0 0" xyz="0 0 0"/>
       <geometry>
-        <mesh filename="package://ernest_description/meshes/pivot.STL"/>
-      </geometry>
-      <material name="">
-        <color rgba="0.752941176470588 0.752941176470588 0.752941176470588 1"/>
-      </material>
-    </visual>
-    <collision>
-      <origin rpy="0 0 0" xyz="0 0 0"/>
-      <geometry>
-        <mesh filename="package://ernest_description/meshes/pivot.STL"/>
+        <mesh filename="package://description/meshes/pivot.STL"/>
+      </geometry>
+      <material name="">
+        <color rgba="0.752941176470588 0.752941176470588 0.752941176470588 1"/>
+      </material>
+    </visual>
+    <collision>
+      <origin rpy="0 0 0" xyz="0 0 0"/>
+      <geometry>
+        <mesh filename="package://description/meshes/pivot.STL"/>
       </geometry>
     </collision>
@@ -68,14 +68,14 @@
       <origin rpy="0 0 0" xyz="0 0 0"/>
       <geometry>
-        <mesh filename="package://ernest_description/meshes/bogie.STL"/>
-      </geometry>
-      <material name="">
-        <color rgba="0.792156862745098 0.819607843137255 0.933333333333333 1"/>
-      </material>
-    </visual>
-    <collision>
-      <origin rpy="0 0 0" xyz="0 0 0"/>
-      <geometry>
-        <mesh filename="package://ernest_description/meshes/bogie.STL"/>
+        <mesh filename="package://description/meshes/bogie.STL"/>
+      </geometry>
+      <material name="">
+        <color rgba="0.792156862745098 0.819607843137255 0.933333333333333 1"/>
+      </material>
+    </visual>
+    <collision>
+      <origin rpy="0 0 0" xyz="0 0 0"/>
+      <geometry>
+        <mesh filename="package://description/meshes/bogie.STL"/>
       </geometry>
     </collision>
@@ -96,14 +96,14 @@
       <origin rpy="0 0 0" xyz="0 0 0"/>
       <geometry>
-        <mesh filename="package://ernest_description/meshes/front_left_steer.STL"/>
-      </geometry>
-      <material name="">
-        <color rgba="0.752941176470588 0.752941176470588 0.752941176470588 1"/>
-      </material>
-    </visual>
-    <collision>
-      <origin rpy="0 0 0" xyz="0 0 0"/>
-      <geometry>
-        <mesh filename="package://ernest_description/meshes/front_left_steer.STL"/>
+        <mesh filename="package://description/meshes/front_left_steer.STL"/>
+      </geometry>
+      <material name="">
+        <color rgba="0.752941176470588 0.752941176470588 0.752941176470588 1"/>
+      </material>
+    </visual>
+    <collision>
+      <origin rpy="0 0 0" xyz="0 0 0"/>
+      <geometry>
+        <mesh filename="package://description/meshes/front_left_steer.STL"/>
       </geometry>
     </collision>
@@ -124,14 +124,14 @@
       <origin rpy="0 0 0" xyz="0 0 0"/>
       <geometry>
-        <mesh filename="package://ernest_description/meshes/front_left_wheel.STL"/>
-      </geometry>
-      <material name="">
-        <color rgba="0.792156862745098 0.819607843137255 0.933333333333333 1"/>
-      </material>
-    </visual>
-    <collision>
-      <origin rpy="0 0 0" xyz="0 0 0"/>
-      <geometry>
-        <mesh filename="package://ernest_description/meshes/front_left_wheel.STL"/>
+        <mesh filename="package://description/meshes/front_left_wheel.STL"/>
+      </geometry>
+      <material name="">
+        <color rgba="0.792156862745098 0.819607843137255 0.933333333333333 1"/>
+      </material>
+    </visual>
+    <collision>
+      <origin rpy="0 0 0" xyz="0 0 0"/>
+      <geometry>
+        <mesh filename="package://description/meshes/front_left_wheel.STL"/>
       </geometry>
     </collision>
@@ -152,14 +152,14 @@
       <origin rpy="0 0 0" xyz="0 0 0"/>
       <geometry>
-        <mesh filename="package://ernest_description/meshes/front_right_steer.STL"/>
-      </geometry>
-      <material name="">
-        <color rgba="0.752941176470588 0.752941176470588 0.752941176470588 1"/>
-      </material>
-    </visual>
-    <collision>
-      <origin rpy="0 0 0" xyz="0 0 0"/>
-      <geometry>
-        <mesh filename="package://ernest_description/meshes/front_right_steer.STL"/>
+        <mesh filename="package://description/meshes/front_right_steer.STL"/>
+      </geometry>
+      <material name="">
+        <color rgba="0.752941176470588 0.752941176470588 0.752941176470588 1"/>
+      </material>
+    </visual>
+    <collision>
+      <origin rpy="0 0 0" xyz="0 0 0"/>
+      <geometry>
+        <mesh filename="package://description/meshes/front_right_steer.STL"/>
       </geometry>
     </collision>
@@ -180,14 +180,14 @@
       <origin rpy="0 0 0" xyz="0 0 0"/>
       <geometry>
-        <mesh filename="package://ernest_description/meshes/front_right_wheel.STL"/>
-      </geometry>
-      <material name="">
-        <color rgba="0.792156862745098 0.819607843137255 0.933333333333333 1"/>
-      </material>
-    </visual>
-    <collision>
-      <origin rpy="0 0 0" xyz="0 0 0"/>
-      <geometry>
-        <mesh filename="package://ernest_description/meshes/front_right_wheel.STL"/>
+        <mesh filename="package://description/meshes/front_right_wheel.STL"/>
+      </geometry>
+      <material name="">
+        <color rgba="0.792156862745098 0.819607843137255 0.933333333333333 1"/>
+      </material>
+    </visual>
+    <collision>
+      <origin rpy="0 0 0" xyz="0 0 0"/>
+      <geometry>
+        <mesh filename="package://description/meshes/front_right_wheel.STL"/>
       </geometry>
     </collision>
@@ -208,14 +208,14 @@
       <origin rpy="0 0 0" xyz="0 0 0"/>
       <geometry>
-        <mesh filename="package://ernest_description/meshes/rear_right_steer.STL"/>
-      </geometry>
-      <material name="">
-        <color rgba="0.752941176470588 0.752941176470588 0.752941176470588 1"/>
-      </material>
-    </visual>
-    <collision>
-      <origin rpy="0 0 0" xyz="0 0 0"/>
-      <geometry>
-        <mesh filename="package://ernest_description/meshes/rear_right_steer.STL"/>
+        <mesh filename="package://description/meshes/rear_right_steer.STL"/>
+      </geometry>
+      <material name="">
+        <color rgba="0.752941176470588 0.752941176470588 0.752941176470588 1"/>
+      </material>
+    </visual>
+    <collision>
+      <origin rpy="0 0 0" xyz="0 0 0"/>
+      <geometry>
+        <mesh filename="package://description/meshes/rear_right_steer.STL"/>
       </geometry>
     </collision>
@@ -236,14 +236,14 @@
       <origin rpy="0 0 0" xyz="0 0 0"/>
       <geometry>
-        <mesh filename="package://ernest_description/meshes/rear_right_wheel.STL"/>
-      </geometry>
-      <material name="">
-        <color rgba="0.792156862745098 0.819607843137255 0.933333333333333 1"/>
-      </material>
-    </visual>
-    <collision>
-      <origin rpy="0 0 0" xyz="0 0 0"/>
-      <geometry>
-        <mesh filename="package://ernest_description/meshes/rear_right_wheel.STL"/>
+        <mesh filename="package://description/meshes/rear_right_wheel.STL"/>
+      </geometry>
+      <material name="">
+        <color rgba="0.792156862745098 0.819607843137255 0.933333333333333 1"/>
+      </material>
+    </visual>
+    <collision>
+      <origin rpy="0 0 0" xyz="0 0 0"/>
+      <geometry>
+        <mesh filename="package://description/meshes/rear_right_wheel.STL"/>
       </geometry>
     </collision>
@@ -264,14 +264,14 @@
       <origin rpy="0 0 0" xyz="0 0 0"/>
       <geometry>
-        <mesh filename="package://ernest_description/meshes/rear_left_steer.STL"/>
-      </geometry>
-      <material name="">
-        <color rgba="0.752941176470588 0.752941176470588 0.752941176470588 1"/>
-      </material>
-    </visual>
-    <collision>
-      <origin rpy="0 0 0" xyz="0 0 0"/>
-      <geometry>
-        <mesh filename="package://ernest_description/meshes/rear_left_steer.STL"/>
+        <mesh filename="package://description/meshes/rear_left_steer.STL"/>
+      </geometry>
+      <material name="">
+        <color rgba="0.752941176470588 0.752941176470588 0.752941176470588 1"/>
+      </material>
+    </visual>
+    <collision>
+      <origin rpy="0 0 0" xyz="0 0 0"/>
+      <geometry>
+        <mesh filename="package://description/meshes/rear_left_steer.STL"/>
       </geometry>
     </collision>
@@ -292,14 +292,14 @@
       <origin rpy="0 0 0" xyz="0 0 0"/>
       <geometry>
-        <mesh filename="package://ernest_description/meshes/rear_left_wheel.STL"/>
-      </geometry>
-      <material name="">
-        <color rgba="0.792156862745098 0.819607843137255 0.933333333333333 1"/>
-      </material>
-    </visual>
-    <collision>
-      <origin rpy="0 0 0" xyz="0 0 0"/>
-      <geometry>
-        <mesh filename="package://ernest_description/meshes/rear_left_wheel.STL"/>
+        <mesh filename="package://description/meshes/rear_left_wheel.STL"/>
+      </geometry>
+      <material name="">
+        <color rgba="0.792156862745098 0.819607843137255 0.933333333333333 1"/>
+      </material>
+    </visual>
+    <collision>
+      <origin rpy="0 0 0" xyz="0 0 0"/>
+      <geometry>
+        <mesh filename="package://description/meshes/rear_left_wheel.STL"/>
       </geometry>
     </collision>
@@ -311,4 +311,5 @@
     <axis xyz="0 0 1"/>
   </joint>
+  <!-- IMU sensor-->
 </xacro:macro>
 </robot>

File: description/urdf/ernest_system.urdf.xacro (robot description, xacro)
@@ -5,9 +5,9 @@
   <xacro:arg name="use_gazebo" default="true" />
   <xacro:arg name="use_lowpoly" default="true" />
-  <xacro:include filename="$(find ernest_description)/urdf/ernest.urdf.xacro" />
-  <xacro:include filename="$(find ernest_description)/urdf/robot_core.urdf.xacro" />
+  <xacro:include filename="$(find description)/urdf/ernest.urdf.xacro" />
+  <xacro:include filename="$(find description)/urdf/robot_core.urdf.xacro" />
   <!-- Import stm ros2_control description -->
-  <xacro:include filename="$(find ernest_description)/urdf/joint_traj_controller.xacro"/>
-  <xacro:include filename="$(find ernest_description)/urdf/ernest_gazebo.xacro" />
+  <xacro:include filename="$(find description)/urdf/joint_traj_controller.xacro"/>
+  <xacro:include filename="$(find description)/urdf/ernest_gazebo.xacro" />
   <xacro:ernest_system
     name="ErnestSystem"

Commit message: made changes

File: description/urdf/ernest.urdf.xacro (robot description, xacro)
@@ -109,5 +109,6 @@
     </collision>
   </link>
-  <joint name="front_left_steer_joint" type="continuous">
+  <joint name="front_left_steer_joint" type="revolute">
+    <limit effort="50" lower="-0.8" upper="0.8" velocity="30"/>
     <origin rpy="-1.5707963267949 0.0208107531087718 0" xyz="0.399593578400315 0.05 0.0507993775470971"/>
     <parent link="bogie"/>
@@ -165,5 +166,6 @@
     </collision>
   </link>
-  <joint name="front_right_steer_joint" type="continuous">
+  <joint name="front_right_steer_joint" type="revolute">
+    <limit effort="50" lower="-0.8" upper="0.8" velocity="30"/>
     <origin rpy="-1.57079632679545 -1.56850410535828 0" xyz="-0.399593578400314 0.05 0.0507993775470972"/>
     <parent link="bogie"/>
@@ -221,5 +223,6 @@
     </collision>
   </link>
-  <joint name="rear_right_steer_joint" type="continuous">
+  <joint name="rear_right_steer_joint" type="revolute">
+    <limit effort="50" lower="-0.8" upper="0.8" velocity="30"/>
     <origin rpy="0 0 0" xyz="0.4038086578651 -0.313808657865102 -0.01666"/>
     <parent link="chassis"/>
@@ -277,5 +280,6 @@
     </collision>
   </link>
-  <joint name="rear_left_steer_joint" type="continuous">
+  <joint name="rear_left_steer_joint" type="revolute">
+    <limit effort="50" lower="-0.8" upper="0.8" velocity="30"/>
     <origin rpy="0 0 -1.56733797587802" xyz="-0.403808657865099 -0.313808657865101 -0.01666"/>
     <parent link="chassis"/>

File: description/urdf/ernest_gazebo.xacro (robot description, xacro)
@@ -16,5 +16,5 @@
       <frame_name>map</frame_name>
       <body_name>base_link</body_name>
-      <update_rate>50.0</update_rate>
+      <update_rate>10.0</update_rate>
       <gaussian_noise>0.01</gaussian_noise>
     </plugin>

File: description/urdf/joint_traj_controller.xacro (robot description, xacro)
@@ -10,6 +10,6 @@
       <joint name="rear_left_steer_joint">
         <command_interface name="position">
-          <param name="min">-1.57</param>
-          <param name="max">1.57</param>
+          <param name="min">-0.8</param>
+          <param name="max">0.8</param>
         </command_interface>
         <state_interface name="position"/>
@@ -18,4 +18,36 @@
       <joint name="rear_right_steer_joint">
         <command_interface name="position">
+          <param name="min">-0.8</param>
+          <param name="max">0.8</param>
+        </command_interface>
+        <state_interface name="position"/>
+        <state_interface name="velocity"/>
+      </joint>
+      <joint name="front_left_steer_joint">
+        <command_interface name="position">
+          <param name="min">-0.8</param>
+          <param name="max">0.8</param>
+        </command_interface>
+        <state_interface name="position"/>
+        <state_interface name="velocity"/>
+      </joint>
+      <joint name="front_right_steer_joint">
+        <command_interface name="position">
+          <param name="min">-0.8</param>
+          <param name="max">0.8</param>
+        </command_interface>
+        <state_interface name="position"/>
+        <state_interface name="velocity"/>
+      </joint>
+      <joint name="pivot_joint">
+        <command_interface name="position">
+          <param name="min">-0.4</param>
+          <param name="max">0.4</param>
+        </command_interface>
+        <state_interface name="position"/>
+        <state_interface name="velocity"/>
+      </joint>
+      <joint name="rear_right_wheel_joint">
+        <command_interface name="velocity">
           <param name="min">-1</param>
           <param name="max">1</param>
@@ -24,40 +56,8 @@
         <state_interface name="velocity"/>
       </joint>
-      <joint name="front_left_steer_joint">
-        <command_interface name="position">
+      <joint name="rear_left_wheel_joint">
+        <command_interface name="velocity">
           <param name="min">-1</param>
           <param name="max">1</param>
-        </command_interface>
-        <state_interface name="position"/>
-        <state_interface name="velocity"/>
-      </joint>
-      <joint name="front_right_steer_joint">
-        <command_interface name="position">
-          <param name="min">-1</param>
-          <param name="max">1</param>
-        </command_interface>
-        <state_interface name="position"/>
-        <state_interface name="velocity"/>
-      </joint>
-      <joint name="pivot_joint">
-        <command_interface name="position">
-          <param name="min">-1.57</param>
-          <param name="max">1.57</param>
-        </command_interface>
-        <state_interface name="position"/>
-        <state_interface name="velocity"/>
-      </joint>
-      <joint name="rear_right_wheel_joint">
-        <command_interface name="velocity">
-          <param name="min">-2</param>
-          <param name="max">2</param>
-        </command_interface>
-        <state_interface name="position"/>
-        <state_interface name="velocity"/>
-      </joint>
-      <joint name="rear_left_wheel_joint">
-        <command_interface name="velocity">
-          <param name="min">--2</param>
-          <param name="max">2</param>
         </command_interface>
         <state_interface name="position"/>

Commit message: added ackermann kin

File: description/urdf/ernest.urdf.xacro (robot description, xacro)
@@ -5,7 +5,7 @@
   </link>
   <joint name="frame_joint" type="fixed">
-    <origin  xyz="0 0 0.4"/>
+    <origin rpy="0 0 ${pi/2}" xyz="0 0 0.4"/>
     <parent link="base_link"/>
-    <child link="chassis"/>
+    <child link="pivot"/>
   </joint>
   <link name="chassis">
@@ -55,6 +55,6 @@
   <joint name="pivot_joint" type="continuous">
     <origin rpy="0 0 3.13911747329568" xyz="0 0.4015 -0.00700000000000001"/>
-    <parent link="chassis"/>
-    <child link="pivot"/>
+    <parent link="pivot"/>
+    <child link="chassis"/>
     <axis xyz="0 0 -1"/>
   </joint>

File: description/urdf/joint_traj_controller.xacro (robot description, xacro)
@@ -64,4 +64,20 @@
         <state_interface name="velocity"/>
       </joint>
+      <joint name="front_right_wheel_joint">
+        <command_interface name="velocity">
+          <param name="min">-1</param>
+          <param name="max">1</param>
+        </command_interface>
+        <state_interface name="position"/>
+        <state_interface name="velocity"/>
+      </joint>
+      <joint name="front_left_wheel_joint">
+        <command_interface name="velocity">
+          <param name="min">-1</param>
+          <param name="max">1</param>
+        </command_interface>
+        <state_interface name="position"/>
+        <state_interface name="velocity"/>
+      </joint>
     </ros2_control>
   </xacro:macro>
