Commit message: added all the model in gazebo and simulated

File: description/urdf/ernest.urdf.xacro (robot description, xacro)
@@ -1,11 +1,12 @@
 <?xml version="1.0" ?>
 <robot xmlns:xacro="http://www.ros.org/wiki/xacro" name="ernest">
+<xacro:include filename="$(find description)/urdf/materials.xacro"/>
 <xacro:macro name="ernest" params="prefix">
   <link name="base_link">
   </link>
   <joint name="frame_joint" type="fixed">
-    <origin rpy="0 0 ${pi/2}" xyz="0 0 0.4"/>
+    <origin rpy="0 0 ${- pi/2}" xyz="-0.4 0 0.4"/>
     <parent link="base_link"/>
-    <child link="pivot"/>
+    <child link="chassis"/>
   </joint>
   <link name="chassis">
@@ -18,14 +19,12 @@
       <origin rpy="0 0 0" xyz="0 0 0"/>
       <geometry>
-        <mesh filename="package://description/meshes/chassis.STL"/>
-      </geometry>
-      <material name="">
-        <color rgba="0.752941176470588 0.752941176470588 0.752941176470588 1"/>
-      </material>
-    </visual>
-    <collision>
-      <origin rpy="0 0 0" xyz="0 0 0"/>
-      <geometry>
-        <mesh filename="package://description/meshes/chassis.STL"/>
+        <mesh filename="$(find description)/meshes/chassis.STL"/>
+      </geometry>
+      <material name="white"/>
+    </visual>
+    <collision>
+      <origin rpy="0 0 0" xyz="0 0 0"/>
+      <geometry>
+        <mesh filename="$(find description)/meshes/chassis.STL"/>
       </geometry>
     </collision>
@@ -40,21 +39,20 @@
       <origin rpy="0 0 0" xyz="0 0 0"/>
       <geometry>
-        <mesh filename="package://description/meshes/pivot.STL"/>
-      </geometry>
-      <material name="">
-        <color rgba="0.752941176470588 0.752941176470588 0.752941176470588 1"/>
-      </material>
-    </visual>
-    <collision>
-      <origin rpy="0 0 0" xyz="0 0 0"/>
-      <geometry>
-        <mesh filename="package://description/meshes/pivot.STL"/>
-      </geometry>
-    </collision>
-  </link>
-  <joint name="pivot_joint" type="continuous">
+        <mesh filename="$(find description)/meshes/pivot.STL"/>
+      </geometry>
+      <material name="black"/>
+    </visual>
+    <collision>
+      <origin rpy="0 0 0" xyz="0 0 0"/>
+      <geometry>
+        <mesh filename="$(find description)/meshes/pivot.STL"/>
+      </geometry>
+    </collision>
+  </link>
+  <joint name="pivot_joint" type="revolute">
+    <limit effort="0.001" lower="-0.8" upper="0.8" velocity="30"/>
     <origin rpy="0 0 3.13911747329568" xyz="0 0.4015 -0.00700000000000001"/>
-    <parent link="pivot"/>
-    <child link="chassis"/>
+    <parent link="chassis"/>
+    <child link="pivot"/>
     <axis xyz="0 0 -1"/>
   </joint>
@@ -68,9 +66,7 @@
       <origin rpy="0 0 0" xyz="0 0 0"/>
       <geometry>
-        <mesh filename="package://description/meshes/bogie.STL"/>
-      </geometry>
-      <material name="">
-        <color rgba="0.792156862745098 0.819607843137255 0.933333333333333 1"/>
-      </material>
+        <mesh filename="$(find description)/meshes/bogie.STL"/>
+      </geometry>
+      <material name="white"/>
     </visual>
     <collision>
@@ -98,7 +94,5 @@
         <mesh filename="package://description/meshes/front_left_steer.STL"/>
       </geometry>
-      <material name="">
-        <color rgba="0.752941176470588 0.752941176470588 0.752941176470588 1"/>
-      </material>
+      <material name="black"/>
     </visual>
     <collision>
@@ -127,7 +121,5 @@
         <mesh filename="package://description/meshes/front_left_wheel.STL"/>
       </geometry>
-      <material name="">
-        <color rgba="0.792156862745098 0.819607843137255 0.933333333333333 1"/>
-      </material>
+      <material name="grey"/>
     </visual>
     <collision>
@@ -136,4 +128,15 @@
         <mesh filename="package://description/meshes/front_left_wheel.STL"/>
       </geometry>
+      <friction>
+        <ode>
+          <mu>100000.0</mu>
+          <mu2>100000.0</mu2>
+        </ode>
+        </friction>
+        <contact>
+          <ode>
+            <min_depth>0.003</min_depth>
+          </ode>
+        </contact>
     </collision>
   </link>
@@ -155,7 +158,5 @@
         <mesh filename="package://description/meshes/front_right_steer.STL"/>
       </geometry>
-      <material name="">
-        <color rgba="0.752941176470588 0.752941176470588 0.752941176470588 1"/>
-      </material>
+      <material name="black"/>
     </visual>
     <collision>
@@ -184,7 +185,16 @@
         <mesh filename="package://description/meshes/front_right_wheel.STL"/>
       </geometry>
-      <material name="">
-        <color rgba="0.792156862745098 0.819607843137255 0.933333333333333 1"/>
-      </material>
+      <friction>
+        <ode>
+          <mu>100000.0</mu>
+          <mu2>100000.0</mu2>
+        </ode>
+        </friction>
+        <contact>
+          <ode>
+            <min_depth>0.003</min_depth>
+          </ode>
+        </contact>
+      <material name="grey"/>
     </visual>
     <collision>
@@ -212,7 +222,5 @@
         <mesh filename="package://description/meshes/rear_right_steer.STL"/>
       </geometry>
-      <material name="">
-        <color rgba="0.752941176470588 0.752941176470588 0.752941176470588 1"/>
-      </material>
+      <material name="black"/>
     </visual>
     <collision>
@@ -241,7 +249,16 @@
         <mesh filename="package://description/meshes/rear_right_wheel.STL"/>
       </geometry>
-      <material name="">
-        <color rgba="0.792156862745098 0.819607843137255 0.933333333333333 1"/>
-      </material>
+      <friction>
+        <ode>
+          <mu>100000.0</mu>
+          <mu2>100000.0</mu2>
+        </ode>
+        </friction>
+        <contact>
+          <ode>
+            <min_depth>0.003</min_depth>
+          </ode>
+        </contact>
+      <material name="grey"/>
     </visual>
     <collision>
@@ -269,7 +286,5 @@
         <mesh filename="package://description/meshes/rear_left_steer.STL"/>
       </geometry>
-      <material name="">
-        <color rgba="0.752941176470588 0.752941176470588 0.752941176470588 1"/>
-      </material>
+      <material name="black"/>
     </visual>
     <collision>
@@ -298,7 +313,16 @@
         <mesh filename="package://description/meshes/rear_left_wheel.STL"/>
       </geometry>
-      <material name="">
-        <color rgba="0.792156862745098 0.819607843137255 0.933333333333333 1"/>
-      </material>
+      <friction>
+        <ode>
+          <mu>100000.0</mu>
+          <mu2>100000.0</mu2>
+        </ode>
+        </friction>
+        <contact>
+          <ode>
+            <min_depth>0.003</min_depth>
+          </ode>
+        </contact>
+      <material name="black"/>
     </visual>
     <collision>
@@ -315,5 +339,4 @@
     <axis xyz="0 0 1"/>
   </joint>
-  <!-- IMU sensor-->
 </xacro:macro>
 </robot>

File: description/urdf/ernest_gazebo.xacro (robot description, xacro)
@@ -16,5 +16,5 @@
       <frame_name>map</frame_name>
       <body_name>base_link</body_name>
-      <update_rate>10.0</update_rate>
+      <update_rate>100.0</update_rate>
       <gaussian_noise>0.01</gaussian_noise>
     </plugin>

Commit message: added scope

File: description/urdf/ernest.urdf.xacro (robot description, xacro)
@@ -19,5 +19,5 @@
       <origin rpy="0 0 0" xyz="0 0 0"/>
       <geometry>
-        <mesh filename="$(find description)/meshes/chassis.STL"/>
+        <mesh filename="package://description/meshes/chassis.STL"/>
       </geometry>
       <material name="white"/>
@@ -26,5 +26,5 @@
       <origin rpy="0 0 0" xyz="0 0 0"/>
       <geometry>
-        <mesh filename="$(find description)/meshes/chassis.STL"/>
+        <mesh filename="package://description/meshes/chassis.STL"/>
       </geometry>
     </collision>
@@ -39,12 +39,12 @@
       <origin rpy="0 0 0" xyz="0 0 0"/>
       <geometry>
-        <mesh filename="$(find description)/meshes/pivot.STL"/>
-      </geometry>
-      <material name="black"/>
-    </visual>
-    <collision>
-      <origin rpy="0 0 0" xyz="0 0 0"/>
-      <geometry>
-        <mesh filename="$(find description)/meshes/pivot.STL"/>
+        <mesh filename="package://description/meshes/pivot.STL"/>
+      </geometry>
+      <material name="black"/>
+    </visual>
+    <collision>
+      <origin rpy="0 0 0" xyz="0 0 0"/>
+      <geometry>
+        <mesh filename="package://description/meshes/pivot.STL"/>
       </geometry>
     </collision>
@@ -66,5 +66,5 @@
       <origin rpy="0 0 0" xyz="0 0 0"/>
       <geometry>
-        <mesh filename="$(find description)/meshes/bogie.STL"/>
+        <mesh filename="package://description/meshes/bogie.STL"/>
       </geometry>
       <material name="white"/>
@@ -324,5 +324,5 @@
           </ode>
         </contact>
-      <material name="black"/>
+      <material name="grey"/>
     </visual>
     <collision>

File: description/urdf/ernest_gazebo.xacro (robot description, xacro)
@@ -20,4 +20,37 @@
     </plugin>
   </gazebo>
+   <gazebo reference="chassis">
+    <material>Gazebo/White</material>
+   </gazebo>
+   <gazebo reference="pivot">
+    <material>Gazebo/DarkGrey</material>
+   </gazebo>
+   <gazebo reference="bogie">
+    <material>Gazebo/White</material>
+   </gazebo>
+   <gazebo reference="front_left_steer">
+    <material>Gazebo/DarkGrey</material>
+   </gazebo>
+   <gazebo reference="rear_left_steer">
+    <material>Gazebo/DarkGrey</material>
+   </gazebo>
+   <gazebo reference="front_right_steer">
+    <material>Gazebo/DarkGrey</material>
+   </gazebo>
+   <gazebo reference="rear_right_steer">
+    <material>Gazebo/DarkGrey</material>
+   </gazebo>
+   <gazebo reference="front_left_wheel">
+    <material>Gazebo/Grey</material>
+   </gazebo>
+   <gazebo reference="front_right_wheel">
+    <material>Gazebo/Grey</material>
+   </gazebo>
+   <gazebo reference="rear_left_wheel">
+    <material>Gazebo/Grey</material>
+   </gazebo>
+   <gazebo reference="rear_right_wheel">
+    <material>Gazebo/Grey</material>
+   </gazebo>
 </xacro:macro>
 </robot>

File: description/urdf/materials.xacro (robot description, xacro)
@@ -2,11 +2,11 @@
 <robot xmlns:xacro="http://www.ros.org/wiki/xacro">
   <material name="black">
-    <color rgba="0.0 0.0 0.0 1.0"/>
+    <color rgba="1.0 1.0 0.3 0.5"/>
   </material>
   <material name="white">
-    <color rgba="1.0 1.0 1.0 1.0"/>
+    <color rgba="1.0 1.0 1.0 0.5"/>
   </material>
   <material name="grey">
-    <color rgba="0.5 0.5 0.5 1.0"/>
+    <color rgba="0.5 0.5 0.5 0.5"/>
   </material>
 </robot>

Commit message: added worlds and friction

File: description/urdf/ernest.urdf.xacro (robot description, xacro)
@@ -77,5 +77,6 @@
     </collision>
   </link>
-  <joint name="bogie_joint" type="continuous">
+  <joint name="bogie_joint" type="revolute">
+    <limit effort="0.001" lower="-1" upper="1" velocity="30"/>
     <origin rpy="1.5707963267949 0.000529942236827729 0" xyz="0 -0.101800622452903 -0.0640000000000083"/>
     <parent link="pivot"/>
@@ -124,19 +125,8 @@
     </visual>
     <collision>
-      <origin rpy="0 0 0" xyz="0 0 0"/>
-      <geometry>
-        <mesh filename="package://description/meshes/front_left_wheel.STL"/>
-      </geometry>
-      <friction>
-        <ode>
-          <mu>100000.0</mu>
-          <mu2>100000.0</mu2>
-        </ode>
-        </friction>
-        <contact>
-          <ode>
-            <min_depth>0.003</min_depth>
-          </ode>
-        </contact>
+      <origin rpy="0 0 0" xyz="0 0 -0.012"/>
+      <geometry>
+          <cylinder length="0.112" radius="0.14" />
+        </geometry>
     </collision>
   </link>
@@ -185,21 +175,10 @@
         <mesh filename="package://description/meshes/front_right_wheel.STL"/>
       </geometry>
-      <friction>
-        <ode>
-          <mu>100000.0</mu>
-          <mu2>100000.0</mu2>
-        </ode>
-        </friction>
-        <contact>
-          <ode>
-            <min_depth>0.003</min_depth>
-          </ode>
-        </contact>
-      <material name="grey"/>
-    </visual>
-    <collision>
-      <origin rpy="0 0 0" xyz="0 0 0"/>
-      <geometry>
-        <mesh filename="package://description/meshes/front_right_wheel.STL"/>
+      <material name="grey"/>
+    </visual>
+    <collision>
+      <origin rpy="0 0 0" xyz="0 0 -0.012"/>
+      <geometry>
+        <cylinder length="0.112" radius="0.14" />
       </geometry>
     </collision>
@@ -249,21 +228,10 @@
         <mesh filename="package://description/meshes/rear_right_wheel.STL"/>
       </geometry>
-      <friction>
-        <ode>
-          <mu>100000.0</mu>
-          <mu2>100000.0</mu2>
-        </ode>
-        </friction>
-        <contact>
-          <ode>
-            <min_depth>0.003</min_depth>
-          </ode>
-        </contact>
-      <material name="grey"/>
-    </visual>
-    <collision>
-      <origin rpy="0 0 0" xyz="0 0 0"/>
-      <geometry>
-        <mesh filename="package://description/meshes/rear_right_wheel.STL"/>
+      <material name="grey"/>
+    </visual>
+    <collision>
+      <origin rpy="0 0 0" xyz="0 0 -0.012"/>
+      <geometry>
+        <cylinder length="0.112" radius="0.14" />
       </geometry>
     </collision>
@@ -313,21 +281,10 @@
         <mesh filename="package://description/meshes/rear_left_wheel.STL"/>
       </geometry>
-      <friction>
-        <ode>
-          <mu>100000.0</mu>
-          <mu2>100000.0</mu2>
-        </ode>
-        </friction>
-        <contact>
-          <ode>
-            <min_depth>0.003</min_depth>
-          </ode>
-        </contact>
-      <material name="grey"/>
-    </visual>
-    <collision>
-      <origin rpy="0 0 0" xyz="0 0 0"/>
-      <geometry>
-        <mesh filename="package://description/meshes/rear_left_wheel.STL"/>
+      <material name="grey"/>
+    </visual>
+    <collision>
+      <origin rpy="0 0 0" xyz="0 0 -0.012"/>
+      <geometry>
+        <cylinder length="0.112" radius="0.14" />
       </geometry>
     </collision>

File: description/urdf/ernest_gazebo.xacro (robot description, xacro)
@@ -19,19 +19,4 @@
       <gaussian_noise>0.01</gaussian_noise>
     </plugin>
-  </gazebo>
-  <gazebo reference="pivot_joint">
-    <provide_feedback>true</provide_feedback>
-    <sensor name="force_torque_sensor" type="force_torque">
-      <always_on>true</always_on>
-      <update_rate>100</update_rate>
-      <visualize>true</visualize>
-      <topic>force_torque</topic>
-      <enable_metrics>true</enable_metrics>
-      <pose>0 0 0 0 0 1.57</pose>
-      <force_torque>
-        <frame>sensor</frame>
-        <measure_direction>child_to_parent</measure_direction>
-      </force_torque>
-    </sensor>
   </gazebo>
   <gazebo reference="chassis">
@@ -57,14 +42,70 @@
   </gazebo>
   <gazebo reference="front_left_wheel">
-  <material>Gazebo/Grey</material>
+    <material>Gazebo/Grey</material>
+    <mu1>1000000.0</mu1>
+    <mu2>1000000.0</mu2>
+    <kp>1000000.0</kp>
+    <kd>100000.0</kd>
+    <slip1>0</slip1>
+    <slip2>0</slip2>
+    <minDepth>0.001</minDepth>
+    <maxVel>0</maxVel>
+    <torsional>
+      <ode>
+        <coefficient>1000</coefficient>
+        <slip>0</slip>
+      </ode>
+    </torsional>
   </gazebo>
   <gazebo reference="front_right_wheel">
-  <material>Gazebo/Grey</material>
+    <material>Gazebo/Grey</material>
+    <mu1>1000000.0</mu1>
+    <mu2>1000000.0</mu2>
+    <kp>1000000.0</kp>
+    <kd>100000.0</kd>
+    <slip1>0</slip1>
+    <slip2>0</slip2>
+    <minDepth>0.001</minDepth>
+    <maxVel>0</maxVel>
+    <torsional>
+      <ode>
+        <coefficient>1000</coefficient>
+        <slip>0</slip>
+      </ode>
+    </torsional>
   </gazebo>
   <gazebo reference="rear_left_wheel">
-  <material>Gazebo/Grey</material>
+    <material>Gazebo/Grey</material>
+    <mu1>1000000.0</mu1>
+    <mu2>1000000.0</mu2>
+    <kp>1000000.0</kp>
+    <kd>100000.0</kd>
+    <slip1>0</slip1>
+    <slip2>0</slip2>
+    <minDepth>0.001</minDepth>
+    <maxVel>0</maxVel>
+    <torsional>
+      <ode>
+        <coefficient>1000</coefficient>
+        <slip>0</slip>
+      </ode>
+    </torsional>
   </gazebo>
   <gazebo reference="rear_right_wheel">
-  <material>Gazebo/Grey</material>
+    <material>Gazebo/Grey</material>
+    <mu1>1000000.0</mu1>
+    <mu2>1000000.0</mu2>
+    <kp>1000000.0</kp>
+    <kd>100000.0</kd>
+    <slip1>0</slip1>
+    <slip2>0</slip2>
+    <minDepth>0.001</minDepth>
+    <maxVel>0</maxVel>
+    <torsional>
+      <ode>
+        <coefficient>1000</coefficient>
+        <slip>0</slip>
+      </ode>
+    </torsional>
   </gazebo>
 </xacro:macro>
