Commit message: fixed the code

File: description/urdf/ernest.urdf.xacro (robot description, xacro)
@@ -2,5 +2,5 @@
 <robot xmlns:xacro="http://www.ros.org/wiki/xacro" name="ernest">
 <xacro:include filename="$(find description)/urdf/materials.xacro"/>
-<xacro:macro name="ernest" params="prefix">
+<xacro:macro name="ernest">
   <link name="base_link">
   </link>

File: description/urdf/ernest_gazebo.xacro (robot description, xacro)
@@ -1,5 +1,5 @@
 <?xml version="1.0"?>
 <robot xmlns:xacro="http://www.ros.org/wiki/xacro">
-<xacro:macro name="ernest_gazebo" params="prefix">
+<xacro:macro name="ernest_gazebo">
   <gazebo>
       <plugin filename="libgazebo_ros2_control.so" name="gazebo_ros2_control">
@@ -17,6 +17,69 @@
       <body_name>base_link</body_name>
       <update_rate>100.0</update_rate>
-      <gaussian_noise>0.01</gaussian_noise>
+      <gaussian_noise>0.0</gaussian_noise>
     </plugin>
+  </gazebo>
+  <gazebo reference="front_left_wheel_joint">
+    <provideFeedback>true</provideFeedback>
+  </gazebo>
+  <gazebo reference="front_right_steer_joint">
+    <provideFeedback>true</provideFeedback>
+  </gazebo>
+  <gazebo reference="front_right_wheel_joint">
+    <provideFeedback>true</provideFeedback>
+  </gazebo>
+  <gazebo reference="rear_right_wheel_joint">
+    <provideFeedback>true</provideFeedback>
+  </gazebo>
+  <gazebo reference="rear_left_wheel_joint">
+    <provideFeedback>true</provideFeedback>
+  </gazebo>
+  <gazebo reference="pivot_joint">
+    <provideFeedback>true</provideFeedback>
+  </gazebo>
+  <!-- The ft_sensor plugin -->
+  <gazebo>
+      <plugin name="fr_wheel_sensor" filename="libgazebo_ros_ft_sensor.so">
+        <ros>
+          <remapping>wrench:=fr_wheel_sensor</remapping>
+        </ros>
+        <joint_name>front_right_wheel_joint</joint_name>
+        <updateRate>1000.0</updateRate>
+      </plugin>
+      <plugin name="fl_wheel_sensor" filename="libgazebo_ros_ft_sensor.so">
+        <ros>
+          <remapping>wrench:=fl_wheel_sensor</remapping>
+        </ros>
+        <joint_name>front_left_wheel_joint</joint_name>
+        <updateRate>1000.0</updateRate>
+      </plugin>
+      <plugin name="rr_wheel_sensor" filename="libgazebo_ros_ft_sensor.so">
+        <ros>
+          <remapping>wrench:=rr_wheel_sensor</remapping>
+        </ros>
+        <joint_name>rear_right_wheel_joint</joint_name>
+        <updateRate>1000.0</updateRate>
+      </plugin>
+      <plugin name="rl_wheel_sensor" filename="libgazebo_ros_ft_sensor.so">
+        <ros>
+          <remapping>wrench:=rl_wheel_sensor</remapping>
+        </ros>
+        <joint_name>rear_left_wheel_joint</joint_name>
+        <updateRate>1000.0</updateRate>
+      </plugin>
+      <plugin name="pivot_sensor" filename="libgazebo_ros_ft_sensor.so">
+        <ros>
+          <remapping>wrench:=pivot_sensor</remapping>
+        </ros>
+        <joint_name>pivot_joint</joint_name>
+        <updateRate>1000.0</updateRate>
+      </plugin>
+      <plugin name="steer_sensor" filename="libgazebo_ros_ft_sensor.so">
+        <ros>
+          <remapping>wrench:=steer_sensor</remapping>
+        </ros>
+        <joint_name>front_right_steer_joint</joint_name>
+        <updateRate>1000.0</updateRate>
+      </plugin>
   </gazebo>
   <gazebo reference="chassis">
@@ -43,10 +106,10 @@
   <gazebo reference="front_left_wheel">
     <material>Gazebo/Grey</material>
-<!--    <mu1>10.0</mu1>
-    <mu2>10.0</mu2>
+    <mu1>30.0</mu1>
+    <mu2>30.0</mu2>
     <kp>10000000.0</kp>
     <kd>1000.0</kd>
-    <slip1>0</slip1>
-    <slip2>0</slip2>
+    <slip1>0.01</slip1>
+    <slip2>0.01</slip2>
     <minDepth>0.00001</minDepth>
     <maxVel>0</maxVel>
@@ -56,14 +119,14 @@
         <slip>0</slip>
       </ode>
-    </torsional> -->
+    </torsional>
   </gazebo>
   <gazebo reference="front_right_wheel">
     <material>Gazebo/Grey</material>
-<!--    <mu1>10.0</mu1>
-    <mu2>10.0</mu2>
+    <mu1>30.0</mu1>
+    <mu2>30.0</mu2>
     <kp>10000000.0</kp>
     <kd>1000.0</kd>
-    <slip1>0</slip1>
-    <slip2>0</slip2>
+    <slip1>0.01</slip1>
+    <slip2>0.01</slip2>
     <minDepth>0.00001</minDepth>
     <maxVel>0</maxVel>
@@ -73,14 +136,14 @@
         <slip>0</slip>
       </ode>
-    </torsional> -->
+    </torsional>
   </gazebo>
   <gazebo reference="rear_left_wheel">
     <material>Gazebo/Grey</material>
-  <!--  <mu1>10.0</mu1>
-    <mu2>10.0</mu2>
+    <mu1>30.0</mu1>
+    <mu2>30.0</mu2>
     <kp>10000000.0</kp>
     <kd>1000.0</kd>
-    <slip1>0</slip1>
-    <slip2>0</slip2>
+    <slip1>0.01</slip1>
+    <slip2>0.01</slip2>
     <minDepth>0.00001</minDepth>
     <maxVel>0</maxVel>
@@ -90,14 +153,14 @@
         <slip>0</slip>
       </ode>
-    </torsional> -->
+    </torsional>
   </gazebo>
   <gazebo reference="rear_right_wheel">
     <material>Gazebo/Grey</material>
-  <!--  <mu1>10.0</mu1>
-    <mu2>10.0</mu2>
+    <mu1>30.0</mu1>
+    <mu2>30.0</mu2>
     <kp>10000000.0</kp>
     <kd>1000.0</kd>
-    <slip1>0</slip1>
-    <slip2>0</slip2>
+    <slip1>0.01</slip1>
+    <slip2>0.01</slip2>
     <minDepth>0.00001</minDepth>
     <maxVel>0</maxVel>
@@ -107,5 +170,5 @@
         <slip>0</slip>
       </ode>
-    </torsional> -->
+    </torsional>
   </gazebo>
 </xacro:macro>

File: description/urdf/ernest_system.urdf.xacro (robot description, xacro)
@@ -1,24 +1,12 @@
 <?xml version="1.0"?>
 <robot xmlns:xacro="http://www.ros.org/wiki/xacro"  name="ernest_system">
-  <!-- Enable setting arguments from the launch file -->
-  <xacro:arg name="use_fake_hardware" default="true" />
-  <xacro:arg name="use_gazebo" default="true" />
-  <xacro:arg name="use_lowpoly" default="true" />
-  <xacro:include filename="$(find description)/urdf/ernest.urdf.xacro" />
-  <xacro:include filename="$(find description)/urdf/robot_core.urdf.xacro" />
-  <!-- Import stm ros2_control description -->
+  <!-- Import model -->
+  <xacro:include filename="$(find description)/urdf/ernest.urdf.xacro"/>
+  <!-- Import controller -->
   <xacro:include filename="$(find description)/urdf/joint_traj_controller.xacro"/>
+  <!-- Import gazebo references + pose -->
   <xacro:include filename="$(find description)/urdf/ernest_gazebo.xacro" />
-  <xacro:ernest_system
-    name="ErnestSystem"
-    use_gazebo="$(arg use_gazebo)"/>
-  <xacro:if value="$(arg use_gazebo)">
-    <xacro:ernest_gazebo prefix=""/>
-  </xacro:if>
-  <xacro:if value="$(arg use_lowpoly)">
-    <xacro:robot_core prefix=""/>
-  </xacro:if>
-  <xacro:unless value="$(arg use_lowpoly)">
-    <xacro:ernest prefix=""/>
-  </xacro:unless>
+  <xacro:ernest_gazebo/>
+  <xacro:ernest/>
+  <xacro:joint_traj_controller/>
 </robot>

File: description/urdf/joint_test.xacro (robot description, xacro)
@@ -1,8 +1,10 @@
 <?xml version="1.0"?>
 <robot xmlns:xacro="http://www.ros.org/wiki/xacro"  name="ernest_controller">
-  <xacro:macro name="joint_traj_controller">
-    <ros2_control name="Joint Control" type="system">
+  <xacro:macro name="ernest_system" params="name  use_gazebo:=^|false ">
+    <ros2_control name="${name}" type="system">
       <hardware>
-          <plugin>gazebo_ros2_control/GazeboSystem</plugin>
+          <xacro:if value="${use_gazebo}">
+            <plugin>gazebo_ros2_control/GazeboSystem</plugin>
+          </xacro:if>
       </hardware>
       <joint name="rear_left_steer_joint">
@@ -62,17 +64,9 @@
         <state_interface name="velocity"/>
       </joint>
-      <joint name="front_right_wheel_joint">
-        <command_interface name="velocity">
-          <param name="min">-1</param>
-          <param name="max">1</param>
-        </command_interface>
+      <joint name="front_left_wheel_joint">
         <state_interface name="position"/>
         <state_interface name="velocity"/>
       </joint>
-      <joint name="front_left_wheel_joint">
-        <command_interface name="velocity">
-          <param name="min">-1</param>
-          <param name="max">1</param>
-        </command_interface>
+      <joint name="front_right_wheel_joint">
         <state_interface name="position"/>
         <state_interface name="velocity"/>

Commit message: added masses and inertias

File: description/urdf/ernest.urdf.xacro (robot description, xacro)
@@ -12,7 +12,8 @@
   <link name="chassis">
     <inertial>
-      <origin rpy="0 0 0" xyz="-1.0298688833211E-06 0.0295380349610433 0"/>
-      <mass value="68.3444673293532"/>
-      <inertia ixx="2.38407014740501" ixy="1.00458083063188E-05" ixz="-9.36310845540363E-07" iyy="2.67178308348484" iyz="0.00251180651218514" izz="4.62433309772227"/>
+      <origin rpy="0 0 0" xyz="0.0 -0.1 0.1"/>
+      <mass value="17.31"/>
+      <inertia ixx="4.1455" ixy="0.0210" ixz="-0.0053"
+      iyy="1.4858" iyz="-0.6295" izz="5.2302"/>
     </inertial>
     <visual>
@@ -33,6 +34,6 @@
     <inertial>
       <origin rpy="0 0 0" xyz="-5.83048022436035E-08 -0.0363481578557913 -0.0534922287892846"/>
-      <mass value="1.21599360090943"/>
-      <inertia ixx="0.00252807022514203" ixy="-4.02004758012849E-10" ixz="-8.09265660814765E-10" iyy="0.0022400253412425" iyz="-0.000203652777557111" izz="0.00252590889130123"/>
+      <mass value="2.82"/>
+      <inertia ixx="0.0045" ixy="0.0" ixz="0.0" iyy="0.0044" iyz="0.0" izz="0.0047"/>
     </inertial>
     <visual>
@@ -51,5 +52,5 @@
   </link>
   <joint name="pivot_joint" type="revolute">
-    <limit effort="0.001" lower="-0.8" upper="0.8" velocity="30"/>
+    <limit effort="5.0" lower="-0.8" upper="0.8" velocity="2"/>
     <origin rpy="0 0 3.13911747329568" xyz="0 0.4015 -0.00700000000000001"/>
     <parent link="chassis"/>
@@ -59,7 +60,8 @@
   <link name="bogie">
     <inertial>
-      <origin rpy="0 0 0" xyz="1.79530299480868E-10 0.107565838050474 0.0507988190707989"/>
-      <mass value="4.63613500742378"/>
-      <inertia ixx="0.0176539151712099" ixy="1.33179894816995E-11" ixz="-1.80130416487432E-08" iyy="0.492085815595167" iyz="-2.75247894551671E-07" izz="0.50573206082967"/>
+      <origin rpy="0 0 0" xyz="0.0 0.15 0.05"/>
+      <mass value="8.475"/>
+      <inertia ixx="0.0454" ixy="0.0" ixz="0.0"
+               iyy="1.2486" iyz="0.0012" izz="1.2830"/>
     </inertial>
     <visual>
@@ -78,5 +80,5 @@
   </link>
   <joint name="bogie_joint" type="revolute">
-    <limit effort="0.001" lower="-1" upper="1" velocity="30"/>
+    <limit effort="1000" lower="-1" upper="1" velocity="30"/>
     <origin rpy="1.5707963267949 0.000529942236827729 0" xyz="0 -0.101800622452903 -0.0640000000000083"/>
     <parent link="pivot"/>
@@ -86,7 +88,7 @@
   <link name="front_left_steer">
     <inertial>
-      <origin rpy="0 0 0" xyz="-0.0214602071785041 -1.63416418175188E-08 -0.170809822421106"/>
-      <mass value="3.15693347082843"/>
-      <inertia ixx="0.00959564325201883" ixy="-6.90245158474706E-10" ixz="0.0016350665333109" iyy="0.0124240240946827" iyz="-1.50731012690546E-09" izz="0.0107772256212113"/>
+      <origin rpy="0 0 0" xyz="0.0 0.0 -0.18"/>
+      <mass value="3.15"/>
+      <inertia ixx="0.0235" ixy="0.0" ixz="0.0034" iyy="0.0311" iyz="-0.0" izz="0.0134"/>
     </inertial>
     <visual>
@@ -113,7 +115,8 @@
   <link name="front_left_wheel">
     <inertial>
-      <origin rpy="0 0 0" xyz="-3.33066907387547E-16 4.05231403988182E-15 -0.0103428040717592"/>
-      <mass value="7.89516360300985"/>
-      <inertia ixx="0.0721255226619386" ixy="5.85469173142172E-18" ixz="-4.01154803819637E-18" iyy="0.0721255226619386" iyz="-7.99937915386961E-18" izz="0.124903964328039"/>
+      <origin rpy="0 0 0" xyz="0.0 0.0 -0.0103428040717592"/>
+      <mass value="2.82"/>
+      <inertia ixx="0.0224" ixy="0.0" ixz="-0.0006"
+              iyy="0.0224" iyz="0.0" izz="0.0337"/>
     </inertial>
     <visual>
@@ -125,8 +128,8 @@
     </visual>
     <collision>
-      <origin rpy="0 0 0" xyz="0 0 -0.012"/>
-      <geometry>
-          <cylinder length="0.112" radius="0.14" />
-        </geometry>
+      <origin rpy="0 0 0" xyz="0 0 0.0"/>
+      <geometry>
+          <mesh filename="package://description/meshes/front_left_wheel.STL"/>
+      </geometry>
     </collision>
   </link>
@@ -139,8 +142,7 @@
   <link name="front_right_steer">
     <inertial>
-      <origin rpy="0 0 0" xyz="-1.52169934430901E-08 0.0214602071253955 -0.170809822376615"/>
-      <mass value="3.15693347612183"/>
-      <inertia ixx="0.0124240240575744" ixy="6.60872662000606E-10" ixz="-1.54947980758551E-09" iyy="0.00959564336065084" iyz="-0.00163506652840397" izz="0.0107772257857585"/>
-    </inertial>
+      <origin rpy="0 0 0" xyz="0.0 0.0 -0.18"/>
+      <mass value="3.15"/>
+      <inertia ixx="0.0331" ixy="0.0" ixz="0.0" iyy="0.0235" iyz="-0.0034" izz="0.0134"/>    </inertial>
     <visual>
       <origin rpy="0 0 0" xyz="0 0 0"/>
@@ -167,6 +169,7 @@
     <inertial>
       <origin rpy="0 0 0" xyz="3.33066907387547E-16 2.77555756156289E-16 -0.0103428040717612"/>
-      <mass value="7.89516360300985"/>
-      <inertia ixx="0.0721255226619385" ixy="-3.46944695195361E-18" ixz="1.11723645742842E-18" iyy="0.0721255226619386" iyz="-2.28698895758661E-20" izz="0.124903964328039"/>
+      <mass value="2.82"/>
+      <inertia ixx="0.0224" ixy="0.0" ixz="-0.0006"
+               iyy="0.0224" iyz="0.0" izz="0.0337"/>
     </inertial>
     <visual>
@@ -178,7 +181,7 @@
     </visual>
     <collision>
-      <origin rpy="0 0 0" xyz="0 0 -0.012"/>
-      <geometry>
-        <cylinder length="0.112" radius="0.14" />
+      <origin rpy="0 0 0" xyz="0 0 0.0"/>
+      <geometry>
+        <mesh filename="package://description/meshes/front_right_wheel.STL"/>
       </geometry>
     </collision>
@@ -192,8 +195,7 @@
   <link name="rear_right_steer">
     <inertial>
-      <origin rpy="0 0 0" xyz="-0.0214599012801062 -0.00011457141843102 -0.175249637742071"/>
-      <mass value="3.15693347239416"/>
-      <inertia ixx="0.00959572392851739" ixy="-1.50985192125477E-05" ixz="0.00163504324230246" iyy="0.0124239434676959" iyz="8.72654557966917E-06" izz="0.0107772257336762"/>
-    </inertial>
+      <origin rpy="0 0 0" xyz="0.0 0.0 -0.18"/>
+      <mass value="3.15"/>
+      <inertia ixx="0.0235" ixy="0.0" ixz="0.0034" iyy="0.0311" iyz="0.0" izz="0.0134"/>    </inertial>
     <visual>
       <origin rpy="0 0 0" xyz="0 0 0"/>
@@ -220,6 +222,7 @@
     <inertial>
       <origin rpy="0 0 0" xyz="2.77555756156289E-17 2.22044604925031E-16 -0.0103428040717601"/>
-      <mass value="7.89516360300985"/>
-      <inertia ixx="0.0721255226619386" ixy="-2.88671200177212E-35" ixz="-5.84667280332668E-51" iyy="0.0721255226619387" iyz="-1.12757025938492E-17" izz="0.124903964328039"/>
+      <mass value="2.82"/>
+      <inertia ixx="0.0224" ixy="0.0" ixz="-0.0006"
+              iyy="0.0224" iyz="0.0" izz="0.0337"/>
     </inertial>
     <visual>
@@ -231,7 +234,7 @@
     </visual>
     <collision>
-      <origin rpy="0 0 0" xyz="0 0 -0.012"/>
-      <geometry>
-        <cylinder length="0.112" radius="0.14" />
+      <origin rpy="0 0 0" xyz="0 0 0.0"/>
+      <geometry>
+        <mesh filename="package://description/meshes/rear_right_wheel.STL"/>
       </geometry>
     </collision>
@@ -245,8 +248,7 @@
   <link name="rear_left_steer">
     <inertial>
-      <origin rpy="0 0 0" xyz="-1.54421406217686E-08 0.0214602071095881 -0.175249637732323"/>
-      <mass value="3.15693347259842"/>
-      <inertia ixx="0.0124240240655924" ixy="6.66699103828725E-10" ixz="-1.54116152780023E-09" iyy="0.00959564333765986" iyz="-0.00163506652927261" izz="0.0107772257496637"/>
-    </inertial>
+      <origin rpy="0 0 0" xyz="0.0 0.0 -0.18"/>
+      <mass value="3.15"/>
+      <inertia ixx="0.0311" ixy="0.0" ixz="0.0" iyy="0.0" iyz="-0.0034" izz="0.0134"/>    </inertial>
     <visual>
       <origin rpy="0 0 0" xyz="0 0 0"/>
@@ -273,6 +275,7 @@
     <inertial>
       <origin rpy="0 0 0" xyz="1.66533453693773E-16 -2.77555756156289E-16 -0.0103428040717607"/>
-      <mass value="7.89516360300985"/>
-      <inertia ixx="0.0721255226619386" ixy="5.20417042793042E-18" ixz="-9.45288769135799E-19" iyy="0.0721255226619386" iyz="-7.73849300611529E-18" izz="0.124903964328039"/>
+      <mass value="2.82"/>
+      <inertia ixx="0.0224" ixy="0.0" ixz="-0.0006"
+              iyy="0.0224" iyz="0.0" izz="0.0337"/>
     </inertial>
     <visual>
@@ -284,7 +287,7 @@
     </visual>
     <collision>
-      <origin rpy="0 0 0" xyz="0 0 -0.012"/>
-      <geometry>
-        <cylinder length="0.112" radius="0.14" />
+      <origin rpy="0 0 0" xyz="0 0 0.0"/>
+      <geometry>
+        <mesh filename="package://description/meshes/rear_left_wheel.STL"/>
       </geometry>
     </collision>

File: description/urdf/ernest_gazebo.xacro (robot description, xacro)
@@ -16,5 +16,5 @@
       <frame_name>map</frame_name>
       <body_name>base_link</body_name>
-      <update_rate>100.0</update_rate>
+      <update_rate>10000.0</update_rate>
       <gaussian_noise>0.0</gaussian_noise>
     </plugin>
@@ -47,4 +47,10 @@
     <provideFeedback>true</provideFeedback>
   </gazebo>
+  <gazebo reference="bogie_joint">
+    <provideFeedback>true</provideFeedback>
+  </gazebo>
+  <gazebo reference="pivot">
+    <provideFeedback>true</provideFeedback>
+  </gazebo>
   <!-- The ft_sensor plugin -->
   <gazebo>
@@ -54,5 +60,5 @@
         </ros>
         <joint_name>front_right_wheel_joint</joint_name>
-        <updateRate>1000.0</updateRate>
+        <updateRate>10.0</updateRate>
       </plugin>
       <plugin name="fl_wheel_sensor" filename="libgazebo_ros_ft_sensor.so">
@@ -61,5 +67,5 @@
         </ros>
         <joint_name>front_left_wheel_joint</joint_name>
-        <updateRate>1000.0</updateRate>
+        <updateRate>10.0</updateRate>
       </plugin>
       <plugin name="rr_wheel_sensor" filename="libgazebo_ros_ft_sensor.so">
@@ -68,5 +74,5 @@
         </ros>
         <joint_name>rear_right_wheel_joint</joint_name>
-        <updateRate>1000.0</updateRate>
+        <updateRate>10.0</updateRate>
       </plugin>
       <plugin name="rl_wheel_sensor" filename="libgazebo_ros_ft_sensor.so">
@@ -75,5 +81,5 @@
         </ros>
         <joint_name>rear_left_wheel_joint</joint_name>
-        <updateRate>1000.0</updateRate>
+        <updateRate>10.0</updateRate>
       </plugin>
       <plugin name="pivot_sensor" filename="libgazebo_ros_ft_sensor.so">
@@ -82,5 +88,5 @@
         </ros>
         <joint_name>pivot_joint</joint_name>
-        <updateRate>1000.0</updateRate>
+        <updateRate>10.0</updateRate>
       </plugin>
       <plugin name="fl_steer_sensor" filename="libgazebo_ros_ft_sensor.so">
@@ -88,27 +94,27 @@
           <remapping>wrench:=fl_steer_sensor</remapping>
         </ros>
-        <joint_name>front_right_steer_joint</joint_name>
-        <updateRate>1000.0</updateRate>
+        <joint_name>front_left_steer_joint</joint_name>
+        <updateRate>10.0</updateRate>
       </plugin>
-        <plugin name="fr_steer_sensor" filename="libgazebo_ros_ft_sensor.so">
+      <plugin name="fr_steer_sensor" filename="libgazebo_ros_ft_sensor.so">
         <ros>
           <remapping>wrench:=fr_steer_sensor</remapping>
         </ros>
         <joint_name>front_right_steer_joint</joint_name>
-        <updateRate>1000.0</updateRate>
+        <updateRate>10.0</updateRate>
       </plugin>
-        <plugin name="rl_steer_sensor" filename="libgazebo_ros_ft_sensor.so">
+      <plugin name="rl_steer_sensor" filename="libgazebo_ros_ft_sensor.so">
         <ros>
           <remapping>wrench:=rl_steer_sensor</remapping>
         </ros>
-        <joint_name>front_right_steer_joint</joint_name>
-        <updateRate>1000.0</updateRate>
+        <joint_name>rear_left_steer_joint</joint_name>
+        <updateRate>10.0</updateRate>
       </plugin>
-        <plugin name="rr_steer_sensor" filename="libgazebo_ros_ft_sensor.so">
+      <plugin name="rr_steer_sensor" filename="libgazebo_ros_ft_sensor.so">
         <ros>
           <remapping>wrench:=rr_steer_sensor</remapping>
         </ros>
-        <joint_name>front_right_steer_joint</joint_name>
-        <updateRate>1000.0</updateRate>
+        <joint_name>rear_right_steer_joint</joint_name>
+        <updateRate>10.0</updateRate>
       </plugin>
   </gazebo>
@@ -136,69 +142,39 @@
   <gazebo reference="front_left_wheel">
     <material>Gazebo/Grey</material>
-    <mu1>30.0</mu1>
-    <mu2>30.0</mu2>
+    <mu1>1.0</mu1>
+    <mu2>1.0</mu2>
+    <fdir1>1 0 0</fdir1>
     <kp>10000000.0</kp>
-    <kd>1000.0</kd>
-    <slip1>0.01</slip1>
-    <slip2>0.01</slip2>
-    <minDepth>0.00001</minDepth>
+    <kd>10.0</kd>
+    <minDepth>0.01</minDepth>
     <maxVel>0</maxVel>
-    <torsional>
-      <ode>
-        <coefficient>10</coefficient>
-        <slip>0</slip>
-      </ode>
-    </torsional>
   </gazebo>
   <gazebo reference="front_right_wheel">
     <material>Gazebo/Grey</material>
-    <mu1>30.0</mu1>
-    <mu2>30.0</mu2>
+    <mu1>1.0</mu1>
+    <mu2>1.0</mu2>
+    <fdir1>1 0 0</fdir1>
     <kp>10000000.0</kp>
-    <kd>1000.0</kd>
-    <slip1>0.01</slip1>
-    <slip2>0.01</slip2>
-    <minDepth>0.00001</minDepth>
+    <kd>10.0</kd>
+    <minDepth>0.01</minDepth>
     <maxVel>0</maxVel>
-    <torsional>
-      <ode>
-        <coefficient>10</coefficient>
-        <slip>0</slip>
-      </ode>
-    </torsional>
   </gazebo>
   <gazebo reference="rear_left_wheel">
     <material>Gazebo/Grey</material>
-    <mu1>30.0</mu1>
-    <mu2>30.0</mu2>
+    <mu1>1.0</mu1>
+    <mu2>1.0</mu2>
     <kp>10000000.0</kp>
-    <kd>1000.0</kd>
-    <slip1>0.01</slip1>
-    <slip2>0.01</slip2>
-    <minDepth>0.00001</minDepth>
+    <kd>10.0</kd>
+    <minDepth>0.01</minDepth>
     <maxVel>0</maxVel>
-    <torsional>
-      <ode>
-        <coefficient>10</coefficient>
-        <slip>0</slip>
-      </ode>
-    </torsional>
   </gazebo>
   <gazebo reference="rear_right_wheel">
     <material>Gazebo/Grey</material>
-    <mu1>30.0</mu1>
-    <mu2>30.0</mu2>
+    <mu1>1.0</mu1>
+    <mu2>1.0</mu2>
     <kp>10000000.0</kp>
-    <kd>1000.0</kd>
-    <slip1>0.01</slip1>
-    <slip2>0.01</slip2>
-    <minDepth>0.00001</minDepth>
+    <kd>10.0</kd>
+    <minDepth>0.01</minDepth>
     <maxVel>0</maxVel>
-    <torsional>
-      <ode>
-        <coefficient>10</coefficient>
-        <slip>0</slip>
-      </ode>
-    </torsional>
   </gazebo>
 </xacro:macro>

File: description/urdf/joint_traj_controller.xacro (robot description, xacro)
@@ -79,6 +79,11 @@
       </joint>
       <joint name="bogie_joint">
+        <command_interface name="position">
+          <param name="min">-100000</param>
+          <param name="max">100000</param>
+        </command_interface>
         <state_interface name="position"/>
         <state_interface name="velocity"/>
+        <state_interface name="effort"/>
       </joint>
     </ros2_control>
