Commit message: set velocity

File: description/urdf/ernest.urdf.xacro (robot description, xacro)
@@ -107,5 +107,5 @@
   </link>
   <joint name="front_left_steer_joint" type="revolute">
-    <limit effort="100" lower="-1.57" upper="1.57" velocity="30"/>
+    <limit effort="100" lower="-${pi}" upper="${pi}" velocity="30"/>
     <origin rpy="-1.5707963267949 0.0208107531087718 0" xyz="0.399593578400315 0.05 0.0507993775470971"/>
     <parent link="bogie"/>
@@ -160,5 +160,5 @@
   </link>
   <joint name="front_right_steer_joint" type="revolute">
-    <limit effort="100" lower="-1.57" upper="1.57" velocity="30"/>
+    <limit effort="100" lower="-${pi}" upper="${pi}" velocity="30"/>
     <origin rpy="-1.57079632679545 -1.56850410535828 0" xyz="-0.399593578400314 0.05 0.0507993775470972"/>
     <parent link="bogie"/>
@@ -213,5 +213,5 @@
   </link>
   <joint name="rear_right_steer_joint" type="revolute">
-    <limit effort="100" lower="-1.57" upper="1.57" velocity="30"/>
+    <limit effort="100" lower="-${pi}" upper="${pi}" velocity="30"/>
     <origin rpy="0 0 0" xyz="0.4038086578651 -0.313808657865102 -0.01666"/>
     <parent link="chassis"/>
@@ -266,5 +266,5 @@
   </link>
   <joint name="rear_left_steer_joint" type="revolute">
-    <limit effort="100" lower="-1.57" upper="1.57" velocity="30"/>
+    <limit effort="100" lower="-${pi}" upper="${pi}" velocity="30"/>
     <origin rpy="0 0 -1.56733797587802" xyz="-0.403808657865099 -0.313808657865101 -0.01666"/>
     <parent link="chassis"/>

File: description/urdf/ernest_gazebo.xacro (robot description, xacro)
@@ -59,5 +59,5 @@
         </ros>
         <joint_name>front_right_wheel_joint</joint_name>
-        <updateRate>10.0</updateRate>
+        <updateRate>1000.0</updateRate>
       </plugin>
       <plugin name="fl_wheel_sensor" filename="libgazebo_ros_ft_sensor.so">
@@ -66,5 +66,5 @@
         </ros>
         <joint_name>front_left_wheel_joint</joint_name>
-        <updateRate>10.0</updateRate>
+        <updateRate>1000.0</updateRate>
       </plugin>
       <plugin name="rr_wheel_sensor" filename="libgazebo_ros_ft_sensor.so">
@@ -73,5 +73,5 @@
         </ros>
         <joint_name>rear_right_wheel_joint</joint_name>
-        <updateRate>10.0</updateRate>
+        <updateRate>1000.0</updateRate>
       </plugin>
       <plugin name="rl_wheel_sensor" filename="libgazebo_ros_ft_sensor.so">
@@ -80,5 +80,5 @@
         </ros>
         <joint_name>rear_left_wheel_joint</joint_name>
-        <updateRate>10.0</updateRate>
+        <updateRate>1000.0</updateRate>
       </plugin>
       <plugin name="pivot_sensor" filename="libgazebo_ros_ft_sensor.so">
@@ -87,5 +87,5 @@
         </ros>
         <joint_name>pivot_joint</joint_name>
-        <updateRate>10.0</updateRate>
+        <updateRate>1000.0</updateRate>
       </plugin>
       <plugin name="fl_steer_sensor" filename="libgazebo_ros_ft_sensor.so">
@@ -94,5 +94,5 @@
         </ros>
         <joint_name>front_left_steer_joint</joint_name>
-        <updateRate>10.0</updateRate>
+        <updateRate>1000.0</updateRate>
       </plugin>
       <plugin name="fr_steer_sensor" filename="libgazebo_ros_ft_sensor.so">
@@ -101,5 +101,5 @@
         </ros>
         <joint_name>front_right_steer_joint</joint_name>
-        <updateRate>10.0</updateRate>
+        <updateRate>1000.0</updateRate>
       </plugin>
       <plugin name="rl_steer_sensor" filename="libgazebo_ros_ft_sensor.so">
@@ -108,5 +108,5 @@
         </ros>
         <joint_name>rear_left_steer_joint</joint_name>
-        <updateRate>10.0</updateRate>
+        <updateRate>1000.0</updateRate>
       </plugin>
       <plugin name="rr_steer_sensor" filename="libgazebo_ros_ft_sensor.so">
@@ -115,5 +115,5 @@
         </ros>
         <joint_name>rear_right_steer_joint</joint_name>
-        <updateRate>10.0</updateRate>
+        <updateRate>1000.0</updateRate>
       </plugin>
   </gazebo>
@@ -141,8 +141,8 @@
   <gazebo reference="front_left_wheel">
     <material>Gazebo/Grey</material>
-    <mu1>2.0</mu1>
-    <mu2>2.0</mu2>
-    <kp>10000000.0</kp>
-    <kd>10.0</kd>
+    <mu1>0.5</mu1>
+    <mu2>0.5</mu2>
+    <kp>100000000.0</kp>
+    <kd>100.0</kd>
     <minDepth>0.01</minDepth>
     <maxVel>0</maxVel>
@@ -150,8 +150,8 @@
   <gazebo reference="front_right_wheel">
     <material>Gazebo/Grey</material>
-    <mu1>2.0</mu1>
-    <mu2>2.0</mu2>
-    <kp>10000000.0</kp>
-    <kd>10.0</kd>
+    <mu1>0.5</mu1>
+    <mu2>0.5</mu2>
+    <kp>100000000.0</kp>
+    <kd>100.0</kd>
     <minDepth>0.01</minDepth>
     <maxVel>0</maxVel>
@@ -159,8 +159,8 @@
   <gazebo reference="rear_left_wheel">
     <material>Gazebo/Grey</material>
-    <mu1>2.0</mu1>
-    <mu2>2.0</mu2>
-    <kp>10000000.0</kp>
-    <kd>10.0</kd>
+    <mu1>0.5</mu1>
+    <mu2>0.5</mu2>
+    <kp>100000000.0</kp>
+    <kd>100.0</kd>
     <minDepth>0.01</minDepth>
     <maxVel>0</maxVel>
@@ -168,8 +168,8 @@
   <gazebo reference="rear_right_wheel">
     <material>Gazebo/Grey</material>
-    <mu1>2.0</mu1>
-    <mu2>2.0</mu2>
-    <kp>10000000.0</kp>
-    <kd>10.0</kd>
+    <mu1>0.5</mu1>
+    <mu2>0.5</mu2>
+    <kp>100000000.0</kp>
+    <kd>100.0</kd>
     <minDepth>0.01</minDepth>
     <maxVel>0</maxVel>

Commit message: fixed singularities + bugs

File: description/urdf/ernest.urdf.xacro (robot description, xacro)
@@ -52,5 +52,5 @@
   </link>
   <joint name="pivot_joint" type="revolute">
-    <limit effort="200.0" lower="-0.8" upper="0.8" velocity="10"/>
+    <limit effort="2000.0" lower="-0.8" upper="0.8" velocity="20"/>
     <origin rpy="0 0 3.13911747329568" xyz="0 0.4015 -0.00700000000000001"/>
     <parent link="chassis"/>

File: description/urdf/ernest_gazebo.xacro (robot description, xacro)
@@ -4,5 +4,5 @@
   <gazebo>
       <plugin filename="libgazebo_ros2_control.so" name="gazebo_ros2_control">
-        <parameters>$(find bringup)/config/position_controller_config.yaml</parameters>
+        <parameters>$(find bringup)/config/effort_controller_config.yaml</parameters>
       </plugin>
   </gazebo>

File: description/urdf/ernest_system.urdf.xacro (robot description, xacro)
@@ -4,9 +4,9 @@
   <xacro:include filename="$(find description)/urdf/ernest.urdf.xacro"/>
   <!-- Import controller -->
-  <xacro:include filename="$(find description)/urdf/position_controller.xacro"/>
+  <xacro:include filename="$(find description)/urdf/effort_controller.xacro"/>
   <!-- Import gazebo references + pose -->
   <xacro:include filename="$(find description)/urdf/ernest_gazebo.xacro" />
   <xacro:ernest_gazebo/>
   <xacro:ernest/>
-  <xacro:position_controller/>
+  <xacro:effort_controller/>
 </robot>

File: description/urdf/position_controller.xacro (robot description, xacro)
@@ -39,13 +39,4 @@
         <state_interface name="velocity"/>
       </joint>
-  <!--
-      <joint name="pivot_joint">
-        <command_interface name="position">
-          <param name="min">-0.4</param>
-          <param name="max">0.4</param>
-        </command_interface>
-        <state_interface name="position"/>
-        <state_interface name="velocity"/>
-      </joint>  -->
       <joint name="rear_right_wheel_joint">
         <command_interface name="velocity">
@@ -80,4 +71,17 @@
         <state_interface name="velocity"/>
       </joint>
+      <joint name="pivot_joint">
+        <command_interface name="position">
+          <param name="min">-0.4</param>
+          <param name="max">0.4</param>
+        </command_interface>
+        <state_interface name="position"/>
+        <state_interface name="velocity"/>
+      </joint>
+      <joint name="bogie_joint">
+        <state_interface name="position"/>
+        <state_interface name="velocity"/>
+        <state_interface name="effort"/>
+      </joint>
     </ros2_control>
   </xacro:macro>
