Commit message: fixind all the code

File: description/urdf/effort_controller.xacro (robot description, xacro)
@@ -1,5 +1,5 @@
 <?xml version="1.0"?>
 <robot xmlns:xacro="http://www.ros.org/wiki/xacro"  name="ernest_controller">
-  <xacro:macro name="effort_joint">
+  <xacro:macro name="effort_controller">
     <ros2_control name="Joint Control" type="system">
       <hardware>

File: description/urdf/ernest.urdf.xacro (robot description, xacro)
@@ -52,5 +52,5 @@
   </link>
   <joint name="pivot_joint" type="revolute">
-    <limit effort="100.0" lower="-0.8" upper="0.8" velocity="10"/>
+    <limit effort="200.0" lower="-0.8" upper="0.8" velocity="10"/>
     <origin rpy="0 0 3.13911747329568" xyz="0 0.4015 -0.00700000000000001"/>
     <parent link="chassis"/>
@@ -135,4 +135,5 @@
   </link>
   <joint name="front_left_wheel_joint" type="continuous">
+    <limit effort="100" velocity="10.0"/>
     <origin rpy="1.57079632679491 0.0288958987838113 1.5707963267949" xyz="0 0 -0.214560184613926"/>
     <parent link="front_left_steer"/>
@@ -188,4 +189,5 @@
   </link>
   <joint name="front_right_wheel_joint" type="continuous">
+    <limit effort="100" velocity="10.0"/>
     <origin rpy="1.5707963267949 1.23836412201798 0" xyz="0 0 -0.214560184613926"/>
     <parent link="front_right_steer"/>
@@ -241,4 +243,5 @@
   </link>
   <joint name="rear_right_wheel_joint" type="continuous">
+    <limit effort="100" velocity="10.0"/>
     <origin rpy="0.0053380848461707 1.5707963267949 0" xyz="0 0 -0.219"/>
     <parent link="rear_right_steer"/>
@@ -294,4 +297,5 @@
   </link>
   <joint name="rear_left_wheel_joint" type="continuous">
+    <limit effort="100" velocity="10.0"/>
     <origin rpy="-1.5707963267949 1.3424366648975 -3.14159265358979" xyz="0 0 -0.219"/>
     <parent link="rear_left_steer"/>

File: description/urdf/ernest_gazebo.xacro (robot description, xacro)
@@ -4,5 +4,5 @@
   <gazebo>
       <plugin filename="libgazebo_ros2_control.so" name="gazebo_ros2_control">
-        <parameters>$(find bringup)/config/effort_controller_config.yaml</parameters>
+        <parameters>$(find bringup)/config/position_controller_config.yaml</parameters>
       </plugin>
   </gazebo>

File: description/urdf/ernest_system.urdf.xacro (robot description, xacro)
@@ -4,9 +4,9 @@
   <xacro:include filename="$(find description)/urdf/ernest.urdf.xacro"/>
   <!-- Import controller -->
-  <xacro:include filename="$(find description)/urdf/effort_joint.xacro"/>
+  <xacro:include filename="$(find description)/urdf/position_controller.xacro"/>
   <!-- Import gazebo references + pose -->
   <xacro:include filename="$(find description)/urdf/ernest_gazebo.xacro" />
   <xacro:ernest_gazebo/>
   <xacro:ernest/>
-  <xacro:effort_joint/>
+  <xacro:position_controller/>
 </robot>

File: description/urdf/position_controller.xacro (robot description, xacro)
@@ -1,5 +1,5 @@
 <?xml version="1.0"?>
 <robot xmlns:xacro="http://www.ros.org/wiki/xacro"  name="ernest_controller">
-  <xacro:macro name="joint_traj_controller">
+  <xacro:macro name="position_controller">
     <ros2_control name="Joint Control" type="system">
       <hardware>
@@ -13,4 +13,5 @@
         <state_interface name="position"/>
         <state_interface name="velocity"/>
+        <state_interface name="effort"/>
       </joint>
       <joint name="rear_right_steer_joint">
@@ -38,4 +39,5 @@
         <state_interface name="velocity"/>
       </joint>
+  <!--
       <joint name="pivot_joint">
         <command_interface name="position">
@@ -45,5 +47,5 @@
         <state_interface name="position"/>
         <state_interface name="velocity"/>
-      </joint>
+      </joint>  -->
       <joint name="rear_right_wheel_joint">
         <command_interface name="velocity">
@@ -78,13 +80,4 @@
         <state_interface name="velocity"/>
       </joint>
-      <joint name="bogie_joint">
-        <command_interface name="position">
-          <param name="min">-100000</param>
-          <param name="max">100000</param>
-        </command_interface>
-        <state_interface name="position"/>
-        <state_interface name="velocity"/>
-        <state_interface name="effort"/>
-      </joint>
     </ros2_control>
   </xacro:macro>

Commit message: fixed plots and kinematics

File: description/urdf/effort_controller.xacro (robot description, xacro)
@@ -78,8 +78,17 @@
         <state_interface name="effort"/>
       </joint>
-      <joint name="pivot_joint">
+      <!--<joint name="pivot_joint">
         <command_interface name="effort">
           <param name="min">-100</param>
           <param name="max">100</param>
+        </command_interface>
+        <state_interface name="position"/>
+        <state_interface name="velocity"/>
+        <state_interface name="effort"/>
+      </joint>    -->
+      <joint name="pivot_joint">
+        <command_interface name="effort">
+          <param name="min">-1</param>
+          <param name="max">1</param>
         </command_interface>
         <state_interface name="position"/>

File: description/urdf/ernest.urdf.xacro (robot description, xacro)
@@ -52,5 +52,5 @@
   </link>
   <joint name="pivot_joint" type="revolute">
-    <limit effort="2000.0" lower="-0.8" upper="0.8" velocity="20"/>
+    <limit effort="2000.0" lower="-0.9" upper="0.9" velocity="20"/>
     <origin rpy="0 0 3.13911747329568" xyz="0 0.4015 -0.00700000000000001"/>
     <parent link="chassis"/>

File: description/urdf/ernest_gazebo.xacro (robot description, xacro)
@@ -141,8 +141,8 @@
   <gazebo reference="front_left_wheel">
     <material>Gazebo/Grey</material>
-    <mu1>0.3</mu1>
-    <mu2>0.3</mu2>
-    <kp>100000000.0</kp>
-    <kd>100.0</kd>
+    <mu1>0.6</mu1>
+    <mu2>0.6</mu2>
+    <kp>10000000000.0</kp>
+    <kd>1000000.0</kd>
     <minDepth>0.005</minDepth>
     <maxVel>0</maxVel>
@@ -150,8 +150,8 @@
   <gazebo reference="front_right_wheel">
     <material>Gazebo/Grey</material>
-    <mu1>0.3</mu1>
-    <mu2>0.3</mu2>
-    <kp>100000000.0</kp>
-    <kd>100.0</kd>
+    <mu1>0.6</mu1>
+    <mu2>0.6</mu2>
+    <kp>10000000000.0</kp>
+    <kd>1000000.0</kd>
     <minDepth>0.005</minDepth>
     <maxVel>0</maxVel>
@@ -159,8 +159,8 @@
   <gazebo reference="rear_left_wheel">
     <material>Gazebo/Grey</material>
-    <mu1>0.3</mu1>
-    <mu2>0.3</mu2>
-    <kp>100000000.0</kp>
-    <kd>100.0</kd>
+    <mu1>0.6</mu1>
+    <mu2>0.6</mu2>
+    <kp>10000000000.0</kp>
+    <kd>1000000.0</kd>
     <minDepth>0.005</minDepth>
     <maxVel>0</maxVel>
@@ -168,8 +168,8 @@
   <gazebo reference="rear_right_wheel">
     <material>Gazebo/Grey</material>
-    <mu1>0.3</mu1>
-    <mu2>0.3</mu2>
-    <kp>100000000.0</kp>
-    <kd>100.0</kd>
+    <mu1>0.6</mu1>
+    <mu2>0.6</mu2>
+    <kp>10000000000.0</kp>
+    <kd>1000000.0</kd>
     <minDepth>0.005</minDepth>
     <maxVel>0</maxVel>

File: description/urdf/position_controller.xacro (robot description, xacro)
@@ -46,4 +46,5 @@
         <state_interface name="position"/>
         <state_interface name="velocity"/>
+        <state_interface name="effort"/>
       </joint>
       <joint name="rear_left_wheel_joint">
@@ -54,4 +55,5 @@
         <state_interface name="position"/>
         <state_interface name="velocity"/>
+        <state_interface name="effort"/>
       </joint>
       <joint name="front_right_wheel_joint">
@@ -62,4 +64,5 @@
         <state_interface name="position"/>
         <state_interface name="velocity"/>
+        <state_interface name="effort"/>
       </joint>
       <joint name="front_left_wheel_joint">
@@ -70,4 +73,5 @@
         <state_interface name="position"/>
         <state_interface name="velocity"/>
+        <state_interface name="effort"/>
       </joint>
       <joint name="pivot_joint">
